File: board.kicad_sch (KiCad schematic)
At the start: 46 parts, among them J1 Conn_01x03, J2 Conn_01x08, J3 Conn_01x03, J4 Conn_02x16_Odd_Even, J5 Conn_01x08, J6 Conn_02x16_Odd_Even, SW1 SW_Push, SW2 SW_Push, U1 Pico, U2 AT24CS04-SSHM, U3 PCF8563T, U4 Pico, U5 DS18B20

Commit message: Add files via upload
Parts:
- added J7, J8: Conn_02x16_Odd_Even, Connector_PinHeader_2.54mm:PinHeader_2x16_P2.54mm_Vertical, symbol Connector_Generic:Conn_02x16_Odd_Even
Connections:
- net GND: now also J7.31 (Pin_31), J7.32 (Pin_32), J8.31 (Pin_31), J8.32 (Pin_32)
- net b15: now reaches U4.21 (GPIO16)
- net b15: now also J7.29 (Pin_29), J7.30 (Pin_30)
- net b14: now reaches U4.22 (GPIO17)
- net b14: now also J7.27 (Pin_27), J7.28 (Pin_28)
- net b13: now reaches U4.24 (GPIO18)
- net b13: now also J7.25 (Pin_25), J7.26 (Pin_26)
- net b12: now reaches U4.25 (GPIO19)
- net b12: now also J7.23 (Pin_23), J7.24 (Pin_24)
- net b11: now reaches U4.26 (GPIO20)
- net b11: now also J7.21 (Pin_21), J7.22 (Pin_22)
- net b10: now reaches U4.27 (GPIO21)
- net b10: now also J7.19 (Pin_19), J7.20 (Pin_20)
- net b9: now reaches U4.29 (GPIO22)
- net b9: now also J7.18 (Pin_18)
- net b8: now reaches U4.31 (GPIO26_ADC0)
- net b8: now also J7.15 (Pin_15), J7.16 (Pin_16)
- net b7: now reaches U4.32 (GPIO27_ADC1)
- net b7: now also J7.13 (Pin_13), J7.14 (Pin_14), J7.17 (Pin_17)
- net b6: now reaches U4.33 (AGND)
- net b6: now also J7.11 (Pin_11), J7.12 (Pin_12)
- net b5: now reaches U4.34 (GPIO28_ADC2)
- net b5: now also J7.10 (Pin_10), J7.9 (Pin_9)
- net b4: now reaches U4.35 (ADC_VREF)
- net b4: now also J7.7 (Pin_7), J7.8 (Pin_8)
- net b3: now reaches U4.37 (3V3_EN)
- net b3: now also J7.5 (Pin_5), J7.6 (Pin_6)
- net b2: now reaches U4.39 (VSYS)
- net b2: now also J7.3 (Pin_3), J7.4 (Pin_4)
- net b1: now reaches U4.40 (VBUS)
- net b1: now also J7.1 (Pin_1), J7.2 (Pin_2)
- net d15: now reaches U1.21 (GPIO16)
- net d15: now also J8.29 (Pin_29), J8.30 (Pin_30)
- net d14: now reaches U1.22 (GPIO17)
- net d14: now also J8.27 (Pin_27), J8.28 (Pin_28)
- net d13: now reaches U1.24 (GPIO18)
- net d13: now also J8.25 (Pin_25), J8.26 (Pin_26)
- net d12: now reaches U1.25 (GPIO19)
- net d12: now also J8.23 (Pin_23), J8.24 (Pin_24)
- net d11: now reaches U1.26 (GPIO20)
- net d11: now also J8.21 (Pin_21), J8.22 (Pin_22)
- net d10: now reaches U1.27 (GPIO21)
- net d10: now also J8.19 (Pin_19), J8.20 (Pin_20)
- net d9: now reaches U1.29 (GPIO22)
- net d9: now also J8.17 (Pin_17), J8.18 (Pin_18)
- net d8: now reaches U1.31 (GPIO26_ADC0)
- net d8: now also J8.15 (Pin_15), J8.16 (Pin_16)
- net d7: now reaches U1.32 (GPIO27_ADC1)
- net d7: now also J8.13 (Pin_13), J8.14 (Pin_14)
- net d6: now reaches U1.33 (AGND)
- net d6: now also J8.11 (Pin_11), J8.12 (Pin_12)
- net d5: now reaches U1.34 (GPIO28_ADC2)
- net d5: now also J8.10 (Pin_10), J8.9 (Pin_9)
- net d4: now reaches U1.35 (ADC_VREF)
- net d4: now also J8.7 (Pin_7), J8.8 (Pin_8)
- net d3: now reaches U1.37 (3V3_EN)
- net d3: now also J8.5 (Pin_5), J8.6 (Pin_6)
- net d2: now reaches U1.39 (VSYS)
- net d2: now also J8.3 (Pin_3), J8.4 (Pin_4)
- net d1: now reaches U1.40 (VBUS)
- net d1: now also J8.1 (Pin_1), J8.2 (Pin_2)
Other:
- note removed: "jakie wyprowadzenia dla kolejnych pinów: VBUS, VSYS? (poza GPIO)"

Commit message: Add files via upload
Parts:
- added BT1: Battery, symbol Device:Battery
- added C1, C2: C, symbol Device:C
- added D12, D13: 1N4148WT, Diode_SMD:D_SOD-523, symbol Diode:1N4148WT
- added J10: Conn_01x03, symbol Connector_Generic:Conn_01x03
- added J9: Conn_01x02_Pin, symbol Connector:Conn_01x02_Pin
- added Y1: Crystal, symbol Device:Crystal
Connections:
- net +3.3V: now also U3.8 (VDD)
- net GND: now also U3.4 (VSS), BT1.2 (-), C1.2, C2.1, Y1.2
- net at U3.1 (OSCI): now also C1.1
- net at U3.2 (OSCO): now also Y1.1
- net at U3.3 (~{INT}): now also J9.1 (Pin_1)
- net SDA: now reaches U3.5 (SDA)
- net SCL: now reaches U3.6 (SCL)
- net at U3.7 (CLKO): now also J9.2 (Pin_2)
- new net: C2.2, D12.1 (K), D13.1 (K)
Other:
- note added: "PCF"
- note added: "RTC"
- moved on the sheet: J3, R1, R14, R2, U2, U3, U5
