File: board_src/board.kicad_sch (KiCad schematic)
At the start: 41 parts, among them J1 Conn_01x03, J2 Conn_01x08, J4 Conn_02x16_Odd_Even, J5 Conn_01x08, J6 Conn_02x16_Odd_Even, J7 Conn_02x16_Odd_Even, J8 Conn_02x16_Odd_Even, SW1 SW_Push, SW2 SW_Push, U1 Pico, U4 Pico

Commit message: Wersja początkowa 9.0
Parts:
- added J3: Conn_01x03, symbol Connector_Generic:Conn_01x03
Connections:
- net +3.3V: now also J3.1 (Pin_1)
- net GND: now also J3.3 (Pin_3)
- new net czujnik temperatury/czujnik temperatury: J3.2 (Pin_2)
Other:
- sheet czujnik temperatury ports: added czujnik temperatury; removed none

Commit message: wersja dodane arkusze hierarchiczne
Parts:
- removed J3: Conn_01x03, symbol Connector_Generic:Conn_01x03
- D1, D2, D3, D4, D5, D6, D7, D8: footprint LED_THT:LED_D3.0mm_FlatTop -> L128GRN2003500000; symbol Device:LED -> L128-GRN2003500000:L128-GRN2003500000; Height (none) -> 0.75; Manufacturer_Name (none) -> Lumileds; Manufacturer_Part_Number (none) -> L128-GRN2003500000; Mouser Part Number (none) -> 997-L128GRN200350000; Mouser Price/Stock (none) -> https://www.mouser.co.uk/ProductDetail/Lumileds/L128-GRN200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
Connections:
- net at D2.1 (A): now also R3.2; no longer J2.7 (Pin_7)
- net at D2.2 (K): now also J2.8 (Pin_8); no longer R4.2
- net at D4.1 (A): now also R5.2; no longer J2.5 (Pin_5)
- net at D4.2 (K): now also J2.6 (Pin_6); no longer R6.2
- net at D7.1 (A): now also R8.2; no longer J2.2 (Pin_2)
- net at D7.2 (K): now also J2.3 (Pin_3); no longer R9.2
- net at D1.1 (A): now also R10.2; no longer J2.8 (Pin_8)
- net at D1.2 (K): now also J2.1 (Pin_1); no longer R3.2
- net at D8.1 (A): now also R9.2; no longer J2.1 (Pin_1)
- net at D8.2 (K): now also J2.2 (Pin_2); no longer R10.2
- net at D6.1 (A): now also R7.2; no longer J2.3 (Pin_3)
- net at D6.2 (K): now also J2.4 (Pin_4); no longer R8.2
- net at D5.1 (A): now also R6.2; no longer J2.4 (Pin_4)
- net at D5.2 (K): now also J2.5 (Pin_5); no longer R7.2
- net at D3.2 (K): now also J2.7 (Pin_7); no longer R5.2
- net at D3.1 (A): now also R4.2; no longer J2.6 (Pin_6)
Other:
- added sheet Gniazdo kart micro SD (microSD.kicad_sch)
- added sheet Potencjometry (potencjometry.kicad_sch)
- added sheet wyświetlacz (wyświetlacz.kicad_sch)
- sheet czujnik temperatury ports: added none; removed czujnik temperatury
- moved on the sheet: R10, R3, R4, R5, R6, R7, R8, R9

Commit message: wersja dodane arkusze hierarchiczne
Connections:
- net +3.3V: now also J7.24 (Pin_24), J7.26 (Pin_26), J7.28 (Pin_28), J7.30 (Pin_30), J7.32 (Pin_32), J8.24 (Pin_24), J8.26 (Pin_26), J8.28 (Pin_28), J8.30 (Pin_30), J8.32 (Pin_32), U1.40 (VBUS), U4.40 (VBUS)
- net GND: now also J7.23 (Pin_23), J7.25 (Pin_25), J7.27 (Pin_27), J7.29 (Pin_29), J8.23 (Pin_23), J8.25 (Pin_25), J8.27 (Pin_27), J8.29 (Pin_29), U1.33 (AGND), U4.33 (AGND); no longer J7.32 (Pin_32), J8.32 (Pin_32)
- net b1: now also U4.37 (3V3_EN); no longer U4.40 (VBUS)
- net b10: now also U4.22 (GPIO17); no longer U4.27 (GPIO21)
- net b2: now also U4.34 (GPIO28_ADC2); no longer U4.39 (VSYS)
- net b3: now also U4.32 (GPIO27_ADC1); no longer U4.37 (3V3_EN)
- net b4: now also U4.31 (GPIO26_ADC0); no longer U4.35 (ADC_VREF)
- net b5: now also U4.29 (GPIO22); no longer U4.34 (GPIO28_ADC2)
- net b6: now also U4.27 (GPIO21); no longer U4.33 (AGND)
- net b7: now also U4.26 (GPIO20); no longer U4.32 (GPIO27_ADC1)
- net b8: now also U4.25 (GPIO19); no longer U4.31 (GPIO26_ADC0)
- net b9: now also U4.24 (GPIO18); no longer U4.29 (GPIO22)
- net d1: now also U1.37 (3V3_EN); no longer U1.40 (VBUS)
- net d10: now also U1.22 (GPIO17); no longer U1.27 (GPIO21)
- net d11: now also U1.21 (GPIO16); no longer U1.26 (GPIO20)
- net d2: now also U1.34 (GPIO28_ADC2); no longer U1.39 (VSYS)
- net d3: now also U1.32 (GPIO27_ADC1); no longer U1.37 (3V3_EN)
- net d4: now also U1.31 (GPIO26_ADC0); no longer U1.35 (ADC_VREF)
- net d5: now also U1.29 (GPIO22); no longer U1.34 (GPIO28_ADC2)
- net d6: now also U1.27 (GPIO21); no longer U1.33 (AGND)
- net d7: now also U1.26 (GPIO20); no longer U1.32 (GPIO27_ADC1)
- net d8: now also U1.25 (GPIO19); no longer U1.31 (GPIO26_ADC0)
- net d9: now also U1.24 (GPIO18); no longer U1.29 (GPIO22)
- net SWCLK: no longer names the net of U4.41 (SWCLK)
- net SWCLK: no longer U1.41 (SWCLK)
- net SWDIO: no longer names the net of U4.43 (SWDIO)
- net SWDIO: no longer U1.43 (SWDIO)
- net b11 renamed MISO
- net MISO: now also U4.21 (GPIO16); no longer U4.26 (GPIO20)
- removed net b12: J7.23 (Pin_23), J7.24 (Pin_24), U4.25 (GPIO19)
- removed net b13: J7.25 (Pin_25), J7.26 (Pin_26), U4.24 (GPIO18)
- removed net b14: J7.27 (Pin_27), J7.28 (Pin_28), U4.22 (GPIO17)
- removed net b15: J7.29 (Pin_29), J7.30 (Pin_30), U4.21 (GPIO16)
- removed net d12: J8.23 (Pin_23), J8.24 (Pin_24), U1.25 (GPIO19)
- removed net d13: J8.25 (Pin_25), J8.26 (Pin_26), U1.24 (GPIO18)
- removed net d14: J8.27 (Pin_27), J8.28 (Pin_28), U1.22 (GPIO17)
- removed net d15: J8.29 (Pin_29), J8.30 (Pin_30), U1.21 (GPIO16)
- no-connect marks 0 -> 8
Other:
- moved on the sheet: J4, J8, SW1, U1

Commit message: wersja dodane arkusze hierarchiczne
Parts:
- removed D10: LED, LED_THT:LED_D5.0mm-4_RGB_Wide_Pins, symbol Device:LED
- removed D11, D9: LED, symbol Device:LED
- removed J1: Conn_01x03, Connector_PinHeader_2.00mm:PinHeader_1x03_P2.00mm_Vertical, symbol Connector_Generic:Conn_01x03
- removed R11, R12, R13: 221, Resistor_SMD:R_0201_0603Metric, symbol Device:R
Connections:
- net b7: no longer J7.17 (Pin_17)
- net b10 renamed CS
- net b8 renamed MOSI
- net b9 renamed SCK
- net SCK: now also J7.17 (Pin_17)
Other:
- added sheet Dioda RGB (rgb.kicad_sch)
- note removed: "RGB"

Commit message: wersja dodane arkusze hierarchiczne
Parts:
- added U3: Pico, RPi_Pico:RPi_Pico_SMD_TH, symbol MCU_RaspberryPi_and_Boards:Pico
- U1, U4: footprint RPi_Pico:RPi_Pico_SMD_TH -> footprints:RPi_Pico_SMD_TH
Changed lines of the file:
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@@
 			)
 		)
-		(property "Footprint" "RPi_Pico:RPi_Pico_SMD_TH"
+		(property "Footprint" "footprints:RPi_Pico_SMD_TH"
 			(at 64.77 50.8 90)
 			(effects
@@
 	)
 	(symbol
+		(lib_id "MCU_RaspberryPi_and_Boards:Pico")
+		(at -25.4 53.34 0)
+		(unit 1)
+		(exclude_from_sim no)
+		(in_bom yes)
+		(on_board yes)
+		(dnp no)
+		(fields_autoplaced yes)
+		(property "Reference" "U3"
+			(at -25.4 21.59 0)
+			(effects
+				(font
+					(size 1.27 1.27)
+				)
+			)
+		)
+		(property "Value" "Pico"
+			(at -25.4 24.13 0)
+			(effects
+				(font
+					(size 1.27 1.27)
+				)
+			)
+		)
+		(property "Footprint" "RPi_Pico:RPi_Pico_SMD_TH"
+			(at -25.4 53.34 90)
+			(effects
+				(font
+					(size 1.27 1.27)
+				)
+				(hide yes)
+			)
+		)
+		(property "Datasheet" ""
+			(at -25.4 53.34 0)
+			(effects
+				(font
+					(size 1.27 1.27)
+				)
+				(hide yes)
+			)
+		)
+		(property "Description" ""
+			(at -25.4 53.34 0)
+			(effects
+				(font
+					(size 1.27 1.27)
+				)
+				(hide yes)
+			)
+		)
+		(pin "6"
+		)
+		(pin "3"
+		)
+		(pin "5"
+		)
+		(pin "1"
+		)
+		(pin "39"
+		)
+		(pin "36"
+		)
+		(pin "33"
+		)
+		(pin "20"
+		)
+		(pin "40"
+		)
+		(pin "38"
+		)
+		(pin "19"
+		)
+		(pin "35"
+		)
+		(pin "8"
+		)
+		(pin "4"
+		)
+		(pin "7"
+		)
+		(pin "9"
+		)
+		(pin "10"
+		)
+		(pin "2"
+		)
+		(pin "11"
+		)
+		(pin "14"
+		)
+		(pin "16"
+		)
+		(pin "13"
+		)
+		(pin "17"
+		)
+		(pin "41"
+		)
+		(pin "15"
+		)
+		(pin "18"
+		)
+		(pin "42"
+		)
+		(pin "43"
+		)
+		(pin "12"
+		)
+		(pin "37"
+		)
+		(pin "34"
+		)
+		(pin "22"
+		)
+		(pin "27"
+		)
+		(pin "21"
+		)
+		(pin "23"
+		)
+		(pin "31"
+		)
+		(pin "32"
+		)
+		(pin "25"
+		)
+		(pin "24"
+		)
+		(pin "29"
+		)
+		(pin "26"
+		)
+		(pin "28"
+		)
+		(pin "30"
+		)
+		(instances
+			(project ""
+				(path "/772e9f49-cfcf-4cf6-843d-0684684f2d4b"
+					(reference "U3")
+					(unit 1)
+				)
+			)
+		)
+	)
+	(symbol
 		(lib_id "Device:R")
 		(at 74.93 106.68 0)
@@
 			)
 		)
-		(property "Footprint" "RPi_Pico:RPi_Pico_SMD_TH"
+		(property "Footprint" "footprints:RPi_Pico_SMD_TH"
 			(at 177.8 52.07 90)
 			(effects

Commit message: wersja dodane USB i port szeregowy
Parts:
- added J1, J16, J17: Conn_01x05, Connector_PinHeader_1.00mm:PinHeader_1x05_P1.00mm_Vertical, symbol Connector_Generic:Conn_01x05
Connections:
- net +3.3V: now also J16.1 (Pin_1), J16.2 (Pin_2), J16.3 (Pin_3), J16.4 (Pin_4), J16.5 (Pin_5)
- net GND: now also J1.1 (Pin_1), J1.2 (Pin_2), J1.3 (Pin_3), J1.4 (Pin_4), J1.5 (Pin_5)
- net RST: now reaches SW2.1, U4.30 (RUN)
- new net +5.0V: J17.1 (Pin_1), J17.2 (Pin_2), J17.3 (Pin_3), J17.4 (Pin_4), J17.5 (Pin_5)
- no-connect marks 8 -> 51
Other:
- added sheet Port USB (portUSB.kicad_sch)
- added sheet Port szeregowy (portszeregowy.kicad_sch)
- moved on the sheet: J4, J7, J8, SW1, U1, U3

Commit message: wersja z przetwornikiem
Parts:
- removed D1, D3, D5, D7: red, L128GRN2003500000, symbol L128-GRN2003500000:L128-GRN2003500000
- removed D2, D4, D6, D8: green, L128GRN2003500000, symbol L128-GRN2003500000:L128-GRN2003500000
- removed J2: Conn_01x08, Connector_PinHeader_2.54mm:PinHeader_1x08_P2.54mm_Vertical, symbol Connector_Generic:Conn_01x08
- removed J4, J6, J7, J8: Conn_02x16_Odd_Even, Connector_PinHeader_2.54mm:PinHeader_2x16_P2.54mm_Vertical, symbol Connector_Generic:Conn_02x16_Odd_Even
- removed R10, R4, R6, R8: 122, Resistor_SMD:R_0201_0603Metric, symbol Device:R
- removed R3, R5, R7, R9: 221, Resistor_SMD:R_0201_0603Metric, symbol Device:R
- added J18, J20, J21, J22: Conn_02x20_Counter_Clockwise, symbol Connector_Generic:Conn_02x20_Counter_Clockwise
- added J6, J8: Conn_01x03, symbol Connector_Generic:Conn_01x03
- added J7: Conn_01x02, symbol Connector_Generic:Conn_01x02
Connections:
- net +3.3V: no longer U1.36 (3V3), U1.40 (VBUS), U4.36 (3V3), U4.40 (VBUS)
- net GND: no longer U1.13 (GND), U1.18 (GND), U1.23 (GND), U1.28 (GND), U1.3 (GND), U1.33 (AGND), U1.38 (GND), U1.42 (GND), U1.8 (GND), U4.13 (GND), U4.18 (GND), U4.23 (GND), U4.28 (GND), U4.3 (GND), U4.33 (AGND), U4.38 (GND), U4.42 (GND), U4.8 (GND)
- net a1: now also J18.1 (Pin_1), J18.40 (Pin_40)
- net a10: now also U4.10 (GPIO7), J18.10 (Pin_10), J18.31 (Pin_31); no longer U4.12 (GPIO9)
- net a11: now also U4.11 (GPIO8), J18.11 (Pin_11), J18.30 (Pin_30); no longer U4.14 (GPIO10)
- net a12: now also U4.12 (GPIO9), J18.12 (Pin_12), J18.29 (Pin_29); no longer U4.15 (GPIO11)
- net a13: now also U4.13 (GND), J18.13 (Pin_13), J18.28 (Pin_28); no longer U4.16 (GPIO12)
- net a14: now also U4.14 (GPIO10), J18.14 (Pin_14), J18.27 (Pin_27); no longer U4.17 (GPIO13)
- net a15: now also U4.15 (GPIO11), J18.15 (Pin_15), J18.26 (Pin_26); no longer U4.19 (GPIO14)
- net a16: now also U4.16 (GPIO12), J18.16 (Pin_16), J18.25 (Pin_25); no longer U4.20 (GPIO15)
- net a2: now also J18.2 (Pin_2), J18.39 (Pin_39)
- net a3: now also U4.3 (GND), J18.3 (Pin_3), J18.38 (Pin_38); no longer U4.4 (GPIO2)
- net a4: now also U4.4 (GPIO2), J18.37 (Pin_37), J18.4 (Pin_4); no longer U4.5 (GPIO3)
- net a5: now also U4.5 (GPIO3), J18.36 (Pin_36), J18.5 (Pin_5); no longer U4.6 (GPIO4)
- net a6: now also U4.6 (GPIO4), J18.35 (Pin_35), J18.6 (Pin_6); no longer U4.7 (GPIO5)
- net a7: now also U4.7 (GPIO5), J18.34 (Pin_34), J18.7 (Pin_7); no longer U4.9 (GPIO6)
- net a8: now also U4.8 (GND), J18.33 (Pin_33), J18.8 (Pin_8); no longer U4.10 (GPIO7)
- net a9: now also U4.9 (GPIO6), J18.32 (Pin_32), J18.9 (Pin_9); no longer U4.11 (GPIO8)
- net b1: now also U4.40 (VBUS), J20.1 (Pin_1), J20.40 (Pin_40); no longer U4.37 (3V3_EN)
- net b2: now also U4.39 (VSYS), J20.2 (Pin_2), J20.39 (Pin_39); no longer U4.34 (GPIO28_ADC2)
- net b3: now also U4.38 (GND), J20.3 (Pin_3), J20.38 (Pin_38); no longer U4.32 (GPIO27_ADC1)
- net b4: now also U4.37 (3V3_EN), J20.37 (Pin_37), J20.4 (Pin_4); no longer U4.31 (GPIO26_ADC0)
- net b5: now also U4.36 (3V3), J20.36 (Pin_36), J20.5 (Pin_5); no longer U4.29 (GPIO22)
- net b6: now also U4.35 (ADC_VREF), J20.35 (Pin_35), J20.6 (Pin_6); no longer U4.27 (GPIO21)
- net b7: now also U4.34 (GPIO28_ADC2), J20.34 (Pin_34), J20.7 (Pin_7); no longer U4.26 (GPIO20)
- net c1: now also J21.1 (Pin_1), J21.40 (Pin_40)
- net c10: now also U1.10 (GPIO7), J21.10 (Pin_10), J21.31 (Pin_31); no longer U1.12 (GPIO9)
- net c11: now also U1.11 (GPIO8), J21.11 (Pin_11), J21.30 (Pin_30); no longer U1.14 (GPIO10)
- net c12: now also U1.12 (GPIO9), J21.12 (Pin_12), J21.29 (Pin_29); no longer U1.15 (GPIO11)
- net c13: now also U1.13 (GND), J21.13 (Pin_13), J21.28 (Pin_28); no longer U1.16 (GPIO12)
- net c14: now also U1.14 (GPIO10), J21.14 (Pin_14), J21.27 (Pin_27); no longer U1.17 (GPIO13)
- net c15: now also U1.15 (GPIO11), J21.15 (Pin_15), J21.26 (Pin_26); no longer U1.19 (GPIO14)
- net c16: now also U1.16 (GPIO12), J21.16 (Pin_16), J21.25 (Pin_25); no longer U1.20 (GPIO15)
- net c2: now also J21.2 (Pin_2), J21.39 (Pin_39)
- net c3: now also U1.3 (GND), J21.3 (Pin_3), J21.38 (Pin_38); no longer U1.4 (GPIO2)
- net c4: now also U1.4 (GPIO2), J21.37 (Pin_37), J21.4 (Pin_4); no longer U1.5 (GPIO3)
- net c5: now also U1.5 (GPIO3), J21.36 (Pin_36), J21.5 (Pin_5); no longer U1.6 (GPIO4)
- net c6: now also U1.6 (GPIO4), J21.35 (Pin_35), J21.6 (Pin_6); no longer U1.7 (GPIO5)
- net c7: now also U1.7 (GPIO5), J21.34 (Pin_34), J21.7 (Pin_7); no longer U1.9 (GPIO6)
- net c8: now also U1.8 (GND), J21.33 (Pin_33), J21.8 (Pin_8); no longer U1.10 (GPIO7)
- net c9: now also U1.9 (GPIO6), J21.32 (Pin_32), J21.9 (Pin_9); no longer U1.11 (GPIO8)
- net d1: now also U1.40 (VBUS), J22.1 (Pin_1), J22.40 (Pin_40); no longer U1.37 (3V3_EN)
- net d10: now also U1.31 (GPIO26_ADC0), J22.10 (Pin_10), J22.31 (Pin_31); no longer U1.22 (GPIO17)
- net d11: now also U1.30 (RUN), J22.11 (Pin_11), J22.30 (Pin_30); no longer U1.21 (GPIO16)
- net d2: now also U1.39 (VSYS), J22.2 (Pin_2), J22.39 (Pin_39); no longer U1.34 (GPIO28_ADC2)
- net d3: now also U1.38 (GND), J22.3 (Pin_3), J22.38 (Pin_38); no longer U1.32 (GPIO27_ADC1)
- net d4: now also U1.37 (3V3_EN), J22.37 (Pin_37), J22.4 (Pin_4); no longer U1.31 (GPIO26_ADC0)
- net d5: now also U1.36 (3V3), J22.36 (Pin_36), J22.5 (Pin_5); no longer U1.29 (GPIO22)
- net d6: now also U1.35 (ADC_VREF), J22.35 (Pin_35), J22.6 (Pin_6); no longer U1.27 (GPIO21)
- net d7: now also U1.34 (GPIO28_ADC2), J22.34 (Pin_34), J22.7 (Pin_7); no longer U1.26 (GPIO20)
- net d8: now also U1.33 (AGND), J22.33 (Pin_33), J22.8 (Pin_8); no longer U1.25 (GPIO19)
- net d9: now also U1.32 (GPIO27_ADC1), J22.32 (Pin_32), J22.9 (Pin_9); no longer U1.24 (GPIO18)
- net at U4.41 (SWCLK): now also J6.3 (Pin_3)
- net at U4.43 (SWDIO): now also J6.1 (Pin_1)
- net at SW1.1: now also J7.1 (Pin_1); no longer U1.30 (RUN)
- net at U1.41 (SWCLK): now also J8.3 (Pin_3)
- net at U1.43 (SWDIO): now also J8.1 (Pin_1)
- net CS renamed b19
- net b19: now also J20.19 (Pin_19), J20.22 (Pin_22)
- net MISO renamed b20
- net b20: now also J20.20 (Pin_20), J20.21 (Pin_21)
- net MOSI renamed b16
- net b16: now also J20.16 (Pin_16), J20.25 (Pin_25)
- net RST: no longer names the net of SW2.1
- net RST: now also J7.2 (Pin_2); no longer U4.30 (RUN)
- net SCK renamed b17
- net b17: now also J20.17 (Pin_17), J20.24 (Pin_24)
- new net: J8.2 (Pin_2), U1.42 (GND)
- new net: J6.2 (Pin_2), U4.42 (GND)
- new net a17: J18.17 (Pin_17), J18.24 (Pin_24), U4.17 (GPIO13)
- new net a18: J18.18 (Pin_18), J18.23 (Pin_23), U4.18 (GND)
- new net a19: J18.19 (Pin_19), J18.22 (Pin_22), U4.19 (GPIO14)
- new net a20: J18.20 (Pin_20), J18.21 (Pin_21), U4.20 (GPIO15)
- new net b10: J20.10 (Pin_10), J20.31 (Pin_31), U4.31 (GPIO26_ADC0)
- new net b11: J20.11 (Pin_11), J20.30 (Pin_30), U4.30 (RUN)
- new net b12: J20.12 (Pin_12), J20.29 (Pin_29), U4.29 (GPIO22)
- new net b13: J20.13 (Pin_13), J20.28 (Pin_28), U4.28 (GND)
- new net b14: J20.14 (Pin_14), J20.27 (Pin_27), U4.27 (GPIO21)
- new net b15: J20.15 (Pin_15), J20.26 (Pin_26), U4.26 (GPIO20)
- new net b18: J20.18 (Pin_18), J20.23 (Pin_23), U4.23 (GND)
- new net b8: J20.33 (Pin_33), J20.8 (Pin_8), U4.33 (AGND)
- new net b9: J20.32 (Pin_32), J20.9 (Pin_9), U4.32 (GPIO27_ADC1)
- new net c17: J21.17 (Pin_17), J21.24 (Pin_24), U1.17 (GPIO13)
- new net c18: J21.18 (Pin_18), J21.23 (Pin_23), U1.18 (GND)
- new net c19: J21.19 (Pin_19), J21.22 (Pin_22), U1.19 (GPIO14)
- new net c20: J21.20 (Pin_20), J21.21 (Pin_21), U1.20 (GPIO15)
- new net d12: J22.12 (Pin_12), J22.29 (Pin_29), U1.29 (GPIO22)
- new net d13: J22.13 (Pin_13), J22.28 (Pin_28), U1.28 (GND)
- new net d14: J22.14 (Pin_14), J22.27 (Pin_27), U1.27 (GPIO21)
- new net d15: J22.15 (Pin_15), J22.26 (Pin_26), U1.26 (GPIO20)
- new net d16: J22.16 (Pin_16), J22.25 (Pin_25), U1.25 (GPIO19)
- new net d17: J22.17 (Pin_17), J22.24 (Pin_24), U1.24 (GPIO18)
- new net d18: J22.18 (Pin_18), J22.23 (Pin_23), U1.23 (GND)
- new net d19: J22.19 (Pin_19), J22.22 (Pin_22), U1.22 (GPIO17)
- new net d20: J22.20 (Pin_20), J22.21 (Pin_21), U1.21 (GPIO16)
- no-connect marks 51 -> 43
Other:
- removed sheet Port szeregowy
- added sheet LED (led.kicad_sch)
- added sheet Przetwornik (przetwornik.kicad_sch)
- note added: "RUN/RST"
- note removed: "LEDS"
- moved on the sheet: J1, J16, J17, SW1, SW2, U1, U4

Commit message: wersja uzupelnione footprinty
Parts:
- removed J5: Conn_01x08, Connector_PinHeader_2.54mm:PinHeader_1x08_P2.54mm_Vertical, symbol Connector_Generic:Conn_01x08
- removed SW10, SW3, SW4, SW5, SW6, SW7, SW8, SW9: ~, Button_Switch_THT:SW_PUSH_6mm, symbol Switch:SW_Push
- removed U3: Pico, RPi_Pico:RPi_Pico_SMD_TH, symbol MCU_RaspberryPi_and_Boards:Pico
- J1, J16, J17: footprint Connector_PinHeader_1.00mm:PinHeader_1x05_P1.00mm_Vertical -> Connector_PinHeader_2.54mm:PinHeader_1x05_P2.54mm_Vertical
- J18, J20, J21, J22: footprint (none) -> Connector_PinHeader_2.54mm:PinHeader_2x20_P2.54mm_Vertical
- J6, J8: footprint (none) -> Connector_PinHeader_2.54mm:PinHeader_1x03_P2.54mm_Vertical
- J7: footprint (none) -> Connector_PinHeader_2.54mm:PinHeader_1x02_P2.54mm_Vertical
Connections:
- no-connect marks 43 -> 0
Other:
- sheet czujnik temperatury renamed Czujnik temperatury
- sheet wyświetlacz renamed Wyświetlacz
- added sheet Przyciski (przyciski.kicad_sch)
- added sheet Wyświetlacz LED (wyswietlaczled.kicad_sch)
- note removed: "przyciski"
