File: board_src/board.kicad_pcb (KiCad board)
At the start: 2 copper layers, 56 parts, among them J1 Conn_01x03, J2 Conn_01x08, J4 Conn_02x16_Odd_Even, J5 Conn_01x08, J6 Conn_02x16_Odd_Even, J7 Conn_02x16_Odd_Even, J8 Conn_02x16_Odd_Even, SW1 SW_Push, SW2 SW_Push, U1 Pico, U2 AT24CS04-SSHM, U3 PCF8563T, U4 Pico, U5 DS18B20

Commit message: wersja dodane arkusze hierarchiczne
Parts:
- added DS1: HC28010-D, footprints:hc28010-d, F.Cu at (213.4, 45.7)
- added IC2: M24C02-WMN6TP, footprints:SOIC127P600X175-8N, F.Cu at (264.0, 70.5)
- added IC3: DS18B20+, footprints:DS18B20, F.Cu at (263.6, 83.2)
- added IC4: LM317T, footprints:TO255P460X1020X2008-3P, F.Cu at (191.4, 160.4)
- added J12: 112J-TDAR-R01, footprints:112JTDARR01, F.Cu at (197.9, 147.8)
- added LS1: BMT0905XH05, footprints:BMT0905XH05, F.Cu at (199.2, 98.6)
- added R15: 10k, Resistor_SMD:R_0201_0603Metric, F.Cu at (261.0, 74.6)
- added R16: 10k, Resistor_SMD:R_0201_0603Metric, F.Cu at (261.0, 76.4)
- added R17: 10k, Resistor_SMD:R_0201_0603Metric, F.Cu at (271.5, 68.1)
- added R18: 10k, Resistor_SMD:R_0201_0603Metric, F.Cu at (271.5, 69.8)
- added R19: 103, Resistor_SMD:R_0201_0603Metric, F.Cu at (261.0, 86.7)
- added U2: MCP4431-xxxx-ST, Package_SO:TSSOP-20_4.4x6.5mm_P0.65mm, F.Cu at (197.8, 106.3)
- D1, D2, D3, D4, D5, D6, D7, D8: footprint LED_THT:LED_D3.0mm_FlatTop -> footprints:L128GRN2003500000
- moved U5 125.1 mm to (144.8, 142.2)
- moved LED1 65.9 mm to (148.1, 127.0)
- moved U3 10.5 mm to (76.2, 15.2)
- moved R3 4.59 mm to (101.8, 139.4)
- moved R4 4.59 mm to (100.0, 139.4)
- moved R5 4.59 mm to (98.3, 139.4)
- moved R6 4.59 mm to (96.5, 139.4)
- moved R7 4.59 mm to (94.8, 139.4)
- moved R8 4.59 mm to (93.0, 139.4)
- moved R9 4.59 mm to (91.3, 139.4)
Connections:
- C1 pad 1: GND -> gnd
- C2 pad 1: GND -> gnd
- D1 pad 1: Net-(D1-K) -> Net-(D1-A)
- D1 pad 2: Net-(D1-A) -> Net-(D1-K)
- D10 pad 2: +3.3V -> 33,V
- D12 pad 2: unconnected-(D12-A-Pad2) -> 3,3V
- D13 pad 2: unconnected-(D13-A-Pad2) -> Net-(BT2-+)
- D2 pad 1: Net-(D2-K) -> Net-(D2-A)
- D2 pad 2: Net-(D2-A) -> Net-(D2-K)
- D3 pad 1: Net-(D3-K) -> Net-(D3-A)
- D3 pad 2: Net-(D3-A) -> Net-(D3-K)
- D4 pad 1: Net-(D4-K) -> Net-(D4-A)
- D4 pad 2: Net-(D4-A) -> Net-(D4-K)
- D5 pad 1: Net-(D5-K) -> Net-(D5-A)
- D5 pad 2: Net-(D5-A) -> Net-(D5-K)
- D6 pad 1: Net-(D6-K) -> Net-(D6-A)
- D6 pad 2: Net-(D6-A) -> Net-(D6-K)
- D7 pad 1: Net-(D7-K) -> Net-(D7-A)
- D7 pad 2: Net-(D7-A) -> Net-(D7-K)
- D8 pad 1: Net-(D8-K) -> Net-(D8-A)
- D8 pad 2: Net-(D8-A) -> Net-(D8-K)
- J2 pad 1: Net-(D8-K) -> Net-(D1-K)
- J2 pad 2: Net-(D7-K) -> Net-(D8-K)
- J2 pad 3: Net-(D6-K) -> Net-(D7-K)
- J2 pad 4: Net-(D5-K) -> Net-(D6-K)
- J2 pad 5: Net-(D4-K) -> Net-(D5-K)
- J2 pad 6: Net-(D3-K) -> Net-(D4-K)
- J2 pad 7: Net-(D2-K) -> Net-(D3-K)
- J2 pad 8: Net-(D1-K) -> Net-(D2-K)
- J7 pad 31: GND -> gnd
- J7 pad 32: GND -> gnd
- J8 pad 31: GND -> gnd
- J8 pad 32: GND -> gnd
- R10 pad 1: +3.3V -> 33,V
- R10 pad 2: Net-(D8-A) -> Net-(D1-A)
- R14 pad 2: Net-(J3-Pin_2) -> /czujnik temperatury/czujnik temperatury
- R3 pad 1: +3.3V -> 33,V
- R3 pad 2: Net-(D1-A) -> Net-(D2-A)
- R4 pad 1: +3.3V -> 33,V
- R4 pad 2: Net-(D2-A) -> Net-(D3-A)
- R5 pad 1: +3.3V -> 33,V
- R5 pad 2: Net-(D3-A) -> Net-(D4-A)
- R6 pad 1: +3.3V -> 33,V
- R6 pad 2: Net-(D4-A) -> Net-(D5-A)
- R7 pad 1: +3.3V -> 33,V
- R7 pad 2: Net-(D5-A) -> Net-(D6-A)
- R8 pad 1: +3.3V -> 33,V
- R8 pad 2: Net-(D6-A) -> Net-(D7-A)
- R9 pad 1: +3.3V -> 33,V
- R9 pad 2: Net-(D7-A) -> Net-(D8-A)
- SW1 pad 2: GND -> gnd
- SW10 pad 1: GND -> gnd
- SW2 pad 2: GND -> gnd
- SW3 pad 1: GND -> gnd
- SW4 pad 1: GND -> gnd
- SW5 pad 1: GND -> gnd
- SW6 pad 1: GND -> gnd
- SW7 pad 1: GND -> gnd
- SW8 pad 1: GND -> gnd
- SW9 pad 1: GND -> gnd
- U1 pad 13: GND -> gnd
- U1 pad 18: GND -> gnd
- U1 pad 23: GND -> gnd
- U1 pad 28: GND -> gnd
- U1 pad 3: GND -> gnd
- U1 pad 36: +3.3V -> 33,V
- U1 pad 38: GND -> gnd
- U1 pad 42: GND -> gnd
- U1 pad 8: GND -> gnd
- U4 pad 13: GND -> gnd
- U4 pad 18: GND -> gnd
- U4 pad 23: GND -> gnd
- U4 pad 28: GND -> gnd
- U4 pad 3: GND -> gnd
- U4 pad 36: +3.3V -> 33,V
- U4 pad 38: GND -> gnd
- U4 pad 42: GND -> gnd
- U4 pad 8: GND -> gnd
- U5 pad 2: Net-(J3-Pin_2) -> /czujnik temperatury/czujnik temperatury

Commit message: wersja dodane arkusze hierarchiczne
Parts:
- added D14: 1N4007, Diode_THT:D_DO-41_SOD81_P10.16mm_Horizontal, F.Cu at (233.7, 160.0)
- moved U2 200.9 mm to (221.0, 130.2)
- moved U3 200.9 mm to (208.3, 129.5)
- moved D12 166.4 mm to (234.2, 106.8)
- moved D13 166.4 mm to (234.2, 109.2)
- moved R10 166.4 mm to (233.6, 122.8)
- moved U2 166.4 mm to (226.1, 117.5)
- moved U3 166.4 mm to (216.6, 104.7)
- moved C1 128.3 mm to (209.1, 114.3)
- moved C1 128.3 mm to (198.9, 118.2)
- moved C2 128.3 mm to (198.9, 121.9)
- moved D12 128.3 mm to (200.0, 109.3)
- moved D13 128.3 mm to (200.0, 111.8)
- moved D10 120.1 mm to (247.1, 121.9)
- moved J1 120.1 mm to (248.5, 132.1)
- moved U5 106.7 mm to (251.5, 142.2)
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Connections:
- C1 pad 1: gnd -> GND
- C2 pad 1: gnd -> GND
- D10 pad 2: 33,V -> +3.3V
- D12 pad 2: 3,3V -> +3.3V
- DS1 pad 1: gnd -> GND
- DS1 pad 11: gnd -> GND
- DS1 pad 12: gnd -> GND
- DS1 pad 13: gnd -> GND
- DS1 pad 14: gnd -> GND
- DS1 pad 8: gnd -> GND
- DS1 pad 9: 3,3V -> +3.3V
- IC2 pad 1: gnd -> GND
- IC2 pad 2: gnd -> GND
- IC2 pad 3: gnd -> GND
- IC2 pad 4: gnd -> GND
- IC2 pad 8: 3,3V -> +3.3V
- IC3 pad 1: gnd -> GND
- IC3 pad 3: 3,3V -> +3.3V
- IC4 pad 2: unconnected-(IC4-OUTPUT-Pad2) -> Net-(D14-A)
- IC4 pad 3: unconnected-(IC4-INPUT-Pad3) -> +7.0V
- J12 pad 1: unconnected-(J12-DAT2-Pad1) -> /Gniazdo kart micro SD/m1
- J12 pad 2: unconnected-(J12-CD/DAT3-Pad2) -> /Gniazdo kart micro SD/m2
- J12 pad 3: unconnected-(J12-CMD-Pad3) -> /Gniazdo kart micro SD/m3
- J12 pad 4: 3,3V -> +3.3V
- J12 pad 5: unconnected-(J12-CLK-Pad5) -> /Gniazdo kart micro SD/m4
- J12 pad 6: gnd -> GND
- J12 pad 7: unconnected-(J12-DAT0-Pad7) -> /Gniazdo kart micro SD/m5
- J12 pad 8: unconnected-(J12-DAT1-Pad8) -> /Gniazdo kart micro SD/m6
- J12 pad CD1: unconnected-(J12-CARD_DETECTION-PadCD1) -> /Gniazdo kart micro SD/m7
- J12 pad G1: gnd -> GND
- J12 pad MP1: gnd -> GND
- J12 pad MP2: gnd -> GND
- J12 pad MP3: gnd -> GND
- J7 pad 21: /b11 -> /MISO
- J7 pad 22: /b11 -> /MISO
- J7 pad 23: /b12 -> GND
- J7 pad 24: /b12 -> +3.3V
- J7 pad 25: /b13 -> GND
- J7 pad 26: /b13 -> +3.3V
- J7 pad 27: /b14 -> GND
- J7 pad 28: /b14 -> +3.3V
- J7 pad 29: /b15 -> GND
- J7 pad 30: /b15 -> +3.3V
- J7 pad 31: gnd -> GND
- J7 pad 32: gnd -> +3.3V
- J8 pad 23: /d12 -> GND
- J8 pad 24: /d12 -> +3.3V
- J8 pad 25: /d13 -> GND
- J8 pad 26: /d13 -> +3.3V
- J8 pad 27: /d14 -> GND
- J8 pad 28: /d14 -> +3.3V
- J8 pad 29: /d15 -> GND
- J8 pad 30: /d15 -> +3.3V
- J8 pad 31: gnd -> GND
- J8 pad 32: gnd -> +3.3V
- LS1 pad 2: 3,3V -> +3.3V
- R10 pad 1: 33,V -> +3.3V
- R15 pad 2: 3,3V -> +3.3V
- R16 pad 2: 3,3V -> +3.3V
- R17 pad 2: 3,3V -> +3.3V
- R18 pad 2: 3,3V -> +3.3V
- R19 pad 2: 3,3V -> +3.3V
- R3 pad 1: 33,V -> +3.3V
- R4 pad 1: 33,V -> +3.3V
- R5 pad 1: 33,V -> +3.3V
- R6 pad 1: 33,V -> +3.3V
- R7 pad 1: 33,V -> +3.3V
- R8 pad 1: 33,V -> +3.3V
- R9 pad 1: 33,V -> +3.3V
- SW1 pad 2: gnd -> GND
- SW10 pad 1: gnd -> GND
- SW2 pad 2: gnd -> GND
- SW3 pad 1: gnd -> GND
- SW4 pad 1: gnd -> GND
- SW5 pad 1: gnd -> GND
- SW6 pad 1: gnd -> GND
- SW7 pad 1: gnd -> GND
- SW8 pad 1: gnd -> GND
- SW9 pad 1: gnd -> GND
- U1 pad 13: gnd -> GND
- U1 pad 18: gnd -> GND
- U1 pad 21: /d15 -> /d11
- U1 pad 22: /d14 -> /d10
- U1 pad 23: gnd -> GND
- U1 pad 24: /d13 -> /d9
- U1 pad 25: /d12 -> /d8
- U1 pad 26: /d11 -> /d7
- U1 pad 27: /d10 -> /d6
- U1 pad 28: gnd -> GND
- U1 pad 29: /d9 -> /d5
- U1 pad 3: gnd -> GND
- U1 pad 31: /d8 -> /d4
- U1 pad 32: /d7 -> /d3
- U1 pad 33: /d6 -> GND
- U1 pad 34: /d5 -> /d2
- U1 pad 35: /d4 -> unconnected-(U1-ADC_VREF-Pad35)_1
- U1 pad 36: 33,V -> +3.3V
- U1 pad 37: /d3 -> /d1
- U1 pad 38: gnd -> GND
- U1 pad 39: /d2 -> unconnected-(U1-VSYS-Pad39)
- U1 pad 40: /d1 -> +3.3V
- U1 pad 41: /SWCLK -> unconnected-(U1-SWCLK-Pad41)
- U1 pad 42: gnd -> GND
- U1 pad 43: /SWDIO -> unconnected-(U1-SWDIO-Pad43)
- U1 pad 8: gnd -> GND
- U2 pad 10: 3,3V -> +3.3V
- U2 pad 11: 3,3V -> +3.3V
- U2 pad 13: gnd -> GND
- U2 pad 8: gnd -> GND
- U4 pad 13: gnd -> GND
- U4 pad 18: gnd -> GND
- U4 pad 21: /b15 -> /MISO
- U4 pad 22: /b14 -> /b10
- U4 pad 23: gnd -> GND
- U4 pad 24: /b13 -> /b9
- U4 pad 25: /b12 -> /b8
- U4 pad 26: /b11 -> /b7
- U4 pad 27: /b10 -> /b6
- U4 pad 28: gnd -> GND
- U4 pad 29: /b9 -> /b5
- U4 pad 3: gnd -> GND
- U4 pad 31: /b8 -> /b4
- U4 pad 32: /b7 -> /b3
- U4 pad 33: /b6 -> GND
- U4 pad 34: /b5 -> /b2
- U4 pad 35: /b4 -> unconnected-(U4-ADC_VREF-Pad35)
- U4 pad 36: 33,V -> +3.3V
- U4 pad 37: /b3 -> /b1
- U4 pad 38: gnd -> GND
- U4 pad 39: /b2 -> unconnected-(U4-VSYS-Pad39)_1
- U4 pad 40: /b1 -> +3.3V
- U4 pad 41: /SWCLK -> unconnected-(U4-SWCLK-Pad41)_1
- U4 pad 42: gnd -> GND
- U4 pad 43: /SWDIO -> unconnected-(U4-SWDIO-Pad43)
- U4 pad 8: gnd -> GND

Commit message: wersja dodane USB i port szeregowy
Parts:
- added J1: Conn_01x05, Connector_PinHeader_1.00mm:PinHeader_1x05_P1.00mm_Vertical, F.Cu at (44.1, 123.0)
- added J15: Conn_01x03, Connector_PinHeader_2.00mm:PinHeader_1x03_P2.00mm_Vertical, F.Cu at (144.8, 84.4)
- added J16: Conn_01x05, Connector_PinHeader_1.00mm:PinHeader_1x05_P1.00mm_Vertical, F.Cu at (47.5, 123.0)
- added J17: Conn_01x05, Connector_PinHeader_1.00mm:PinHeader_1x05_P1.00mm_Vertical, F.Cu at (50.8, 123.0)
- added J18: TC2050, Connector:Tag-Connect_TC2050-IDC-NL_2x05_P1.27mm_Vertical, F.Cu at (156.2, 59.4)
- added LED1: ASMT-YTB2-0BB02, footprints:ASMT-YTC7-0AA02, F.Cu at (151.5, 87.4)
- added R21: 221, Resistor_SMD:R_0201_0603Metric, F.Cu at (157.1, 72.7)
- added R22: 221, Resistor_SMD:R_0201_0603Metric, F.Cu at (157.5, 74.6)
- added R23: 221, Resistor_SMD:R_0201_0603Metric, F.Cu at (157.5, 76.3)
- U1, U4: footprint RPi_Pico:RPi_Pico_SMD_TH -> footprints:RPi_Pico_SMD_TH
Connections:
- net /MISO renamed MISO
- net /b10 renamed CS
- net /b8 renamed MOSI
- net Net-(U4-RUN) renamed RST
- J7 pad 17: /b7 -> SCK
- J7 pad 18: /b9 -> SCK
- U4 pad 24: /b9 -> SCK

Commit message: wersja z przetwornikiem
Parts:
- removed the C1 at (209.1, 114.3)
- removed the C1 at (198.9, 118.2)
- removed D10: LED, LED_THT:LED_D5.0mm-4_RGB_Wide_Pins
- removed the D12 at (200.0, 109.3)
- removed the D12 at (234.2, 106.8)
- removed the D13 at (200.0, 111.8)
- removed the D13 at (234.2, 109.2)
- removed the J1 at (248.5, 132.1)
- removed the J1 at (44.1, 123.0)
- removed J18: TC2050, Connector:Tag-Connect_TC2050-IDC-NL_2x05_P1.27mm_Vertical
- removed the LED1 at (237.5, 127.0)
- removed the LED1 at (151.5, 87.4)
- removed R11, R12, R13: 221, Resistor_SMD:R_0201_0603Metric
- removed the U2 at (226.1, 117.5)
- removed the U2 at (221.0, 130.2)
- removed the U2 at (264.5, 134.3)
- removed U3 (x2): PCF8563T, Package_SO:SOIC-8_3.9x4.9mm_P1.27mm
- removed U5 (x2): DS18B20, Package_TO_SOT_THT:TO-92_Inline
- added C1: C, Capacitor_SMD:C_0201_0603Metric, F.Cu at (72.6, 119.0)
- added D12: 1N4148WT, Diode_SMD:D_SOD-523, F.Cu at (75.6, 119.4)
- added D13: 1N4148WT, Diode_SMD:D_SOD-523, F.Cu at (75.6, 121.8)
- added IC1: PCF8563TS_4,118, footprints:SOP65P490X110-8N, F.Cu at (49.6, 111.5)
- added IC5: MCP3202-CI_MS, footprints:SOP65P490X110-8N, F.Cu at (49.6, 105.0)
- added J1: Conn_01x05, Connector_PinHeader_1.00mm:PinHeader_1x05_P1.00mm_Vertical, F.Cu at (35.6, 126.6)
- added LED1: ASMT-YTB2-0BB02, footprints:ASMT-YTC7-0AA02, F.Cu at (77.4, 111.9)
- added U2: MCP4431-xxxx-ST, Package_SO:TSSOP-20_4.4x6.5mm_P0.65mm, F.Cu at (91.4, 96.8)
- moved R10 217.2 mm to (18.7, 91.4)
- moved J12 210.9 mm to (68.7, 91.1)
- moved DS1 208.6 mm to (45.9, 170.2)
- moved IC4 184.1 mm to (76.1, 103.8)
- moved D14 182.4 mm to (60.7, 102.1)
- moved LS1 158.1 mm to (92.8, 89.1)
- moved R17 157.2 mm to (72.6, 122.5)
- moved R18 157.2 mm to (72.6, 124.3)
- moved SW10 137.3 mm to (25.4, 121.8)
- moved R15 137.0 mm to (85.1, 115.5)
- moved R16 137.0 mm to (85.1, 117.3)
- moved IC2 137.0 mm to (88.2, 111.4)
- moved IC3 130.4 mm to (98.3, 112.0)
- moved R19 130.4 mm to (95.6, 115.5)
- moved SW9 128.5 mm to (25.4, 113.3)
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Connections:
- SW1 pad 1: Net-(U1-RUN) -> Net-(J7-Pin_1)
- SW2 pad 1: RST -> Net-(J7-Pin_2)
- U1 pad 10: /c8 -> /c10
- U1 pad 11: /c9 -> /c11
- U1 pad 12: /c10 -> /c12
- U1 pad 13: GND -> /c13
- U1 pad 14: /c11 -> /c14
- U1 pad 15: /c12 -> /c15
- U1 pad 16: /c13 -> /c16
- U1 pad 17: /c14 -> /c17
- U1 pad 18: GND -> /c18
- U1 pad 19: /c15 -> /c19
- U1 pad 20: /c16 -> /c20
- U1 pad 21: /d11 -> /d20
- U1 pad 22: /d10 -> /d19
- U1 pad 23: GND -> /d18
- U1 pad 24: /d9 -> /d17
- U1 pad 25: /d8 -> /d16
- U1 pad 26: /d7 -> /d15
- U1 pad 27: /d6 -> /d14
- U1 pad 28: GND -> /d13
- U1 pad 29: /d5 -> /d12
- U1 pad 3: GND -> /c3
- U1 pad 30: Net-(U1-RUN) -> /d11
- U1 pad 31: /d4 -> /d10
- U1 pad 32: /d3 -> /d9
- U1 pad 33: GND -> /d8
- U1 pad 34: /d2 -> /d7
- U1 pad 35: unconnected-(U1-ADC_VREF-Pad35) -> /d6
- U1 pad 36: +3.3V -> /d5
- U1 pad 37: /d1 -> /d4
- U1 pad 38: GND -> /d3
- U1 pad 39: unconnected-(U1-VSYS-Pad39)_1 -> /d2
- U1 pad 4: /c3 -> /c4
- U1 pad 40: +3.3V -> /d1
- U1 pad 41: unconnected-(U1-SWCLK-Pad41) -> Net-(J8-Pin_3)
- U1 pad 42: GND -> Net-(J8-Pin_2)
- U1 pad 43: unconnected-(U1-SWDIO-Pad43)_1 -> Net-(J8-Pin_1)
- U1 pad 5: /c4 -> /c5
- U1 pad 6: /c5 -> /c6
- U1 pad 7: /c6 -> /c7
- U1 pad 8: GND -> /c8
- U1 pad 9: /c7 -> /c9
- U4 pad 10: /a8 -> /a10
- U4 pad 11: /a9 -> /a11
- U4 pad 12: /a10 -> /a12
- U4 pad 13: GND -> /a13
- U4 pad 14: /a11 -> /a14
- U4 pad 15: /a12 -> /a15
- U4 pad 16: /a13 -> /a16
- U4 pad 17: /a14 -> /a17
- U4 pad 18: GND -> /a18
- U4 pad 19: /a15 -> /a19
- U4 pad 20: /a16 -> /a20
- U4 pad 21: MISO -> /b20
- U4 pad 22: CS -> /b19
- U4 pad 23: GND -> /b18
- U4 pad 24: SCK -> /b17
- U4 pad 25: MOSI -> /b16
- U4 pad 26: /b7 -> /b15
- U4 pad 27: /b6 -> /b14
- U4 pad 28: GND -> /b13
- U4 pad 29: /b5 -> /b12
- U4 pad 3: GND -> /a3
- U4 pad 30: RST -> /b11
- U4 pad 31: /b4 -> /b10
- U4 pad 32: /b3 -> /b9
- U4 pad 33: GND -> /b8
- U4 pad 34: /b2 -> /b7
- U4 pad 35: unconnected-(U4-ADC_VREF-Pad35)_1 -> /b6
- U4 pad 36: +3.3V -> /b5
- U4 pad 37: /b1 -> /b4
- U4 pad 38: GND -> /b3
- U4 pad 39: unconnected-(U4-VSYS-Pad39)_1 -> /b2
- U4 pad 4: /a3 -> /a4
- U4 pad 40: +3.3V -> /b1
- U4 pad 41: unconnected-(U4-SWCLK-Pad41)_1 -> Net-(J6-Pin_3)
- U4 pad 42: GND -> Net-(J6-Pin_2)
- U4 pad 43: unconnected-(U4-SWDIO-Pad43) -> Net-(J6-Pin_1)
- U4 pad 5: /a4 -> /a5
- U4 pad 6: /a5 -> /a6
- U4 pad 7: /a6 -> /a7
- U4 pad 8: GND -> /a8
- U4 pad 9: /a7 -> /a9

Commit message: wersja uzupelnione footprinty
Parts:
- added BT2: 502-3, footprints:podstawka_bateria, F.Cu at (137.1, 142.7)
- added C3: 1n, Capacitor_SMD:C_0201_0603Metric, F.Cu at (157.1, 80.3)
- added C4: 100n, Capacitor_SMD:C_1808_4520Metric, F.Cu at (148.9, 71.9)
- added DS2: CA56-21SURKWA, footprints:wyswietlacz7x4, F.Cu at (96.1, 106.5)
- added J10: Conn_01x01_Pin, Connector_PinHeader_2.54mm:PinHeader_1x01_P2.54mm_Vertical, F.Cu at (147.4, 27.5)
- added J11: Conn_01x03, Connector_PinHeader_2.54mm:PinHeader_1x03_P2.54mm_Vertical, F.Cu at (95.7, 143.1)
- added J13: Conn_01x03, Connector_PinHeader_2.54mm:PinHeader_1x13_P2.54mm_Vertical, F.Cu at (157.5, 132.1)
- added J14: Conn_01x07, Connector_PinHeader_2.54mm:PinHeader_1x07_P2.54mm_Vertical, F.Cu at (111.9, 45.4)
- added J18: Conn_02x20_Counter_Clockwise, Connector_PinHeader_2.54mm:PinHeader_2x20_P2.54mm_Vertical, F.Cu at (64.9, 89.2)
- added J19: USB_C_Receptacle_PowerOnly_6P, Connector_USB:USB_C_Receptacle_GCT_USB4135-GF-A_6P_TopMnt_Horizontal, F.Cu at (116.6, 79.6)
- added J20: Conn_02x20_Counter_Clockwise, Connector_PinHeader_2.54mm:PinHeader_2x20_P2.54mm_Vertical, F.Cu at (72.1, 89.2)
- added J21: Conn_02x20_Counter_Clockwise, Connector_PinHeader_2.54mm:PinHeader_2x20_P2.54mm_Vertical, F.Cu at (79.3, 89.2)
- added J22: Conn_02x20_Counter_Clockwise, Connector_PinHeader_2.54mm:PinHeader_2x20_P2.54mm_Vertical, F.Cu at (86.5, 89.2)
- added J23: Conn_01x04, Connector_PinHeader_2.54mm:PinHeader_1x04_P2.54mm_Vertical, F.Cu at (143.0, 67.7)
- added J24: Conn_01x08, Connector_PinHeader_2.54mm:PinHeader_1x08_P2.54mm_Vertical, F.Cu at (116.3, 89.2)
- added J25: Conn_01x04, Connector_PinHeader_2.54mm:PinHeader_1x04_P2.54mm_Vertical, F.Cu at (120.9, 89.2)
- added J3: Conn_01x06, Connector_PinHeader_2.54mm:PinHeader_1x06_P2.54mm_Vertical, F.Cu at (16.8, 69.9)
- added J9: Conn_01x02_Pin, Connector_PinHeader_2.54mm:PinHeader_1x02_P2.54mm_Vertical, F.Cu at (134.9, 156.1)
- added Q1: NPN, Transistor_Power:GaN_Systems_GaNPX-3_5x6.6mm_Drain2.93x0.6mm, F.Cu at (158.6, 122.1)
- added Q2: SS8550, Package_TO_SOT_SMD:SOT-23, F.Cu at (116.4, 111.7)
- added Q3: SS8550, Package_TO_SOT_SMD:SOT-23, F.Cu at (116.4, 116.3)
- added Q4: SS8550, Package_TO_SOT_SMD:SOT-23, F.Cu at (116.4, 121.0)
- added Q5: SS8550, Package_TO_SOT_SMD:SOT-23, F.Cu at (116.4, 125.6)
- added R11: 5.1k, Resistor_SMD:R_0201_0603Metric, F.Cu at (157.1, 82.1)
- added R12: 5.1k, Resistor_SMD:R_0201_0603Metric, F.Cu at (157.1, 83.8)
- added R13: 221, Resistor_SMD:R_0201_0603Metric, F.Cu at (115.2, 128.7)
- added R20: R, Resistor_SMD:R_0201_0603Metric, F.Cu at (139.4, 121.9)
- added R24: 221, Resistor_SMD:R_0201_0603Metric, F.Cu at (115.2, 130.4)
- added R25: 221, Resistor_SMD:R_0201_0603Metric, F.Cu at (115.2, 132.2)
- added R26: 221, Resistor_SMD:R_0201_0603Metric, F.Cu at (115.2, 133.9)
- added R27: 221, Resistor_SMD:R_0201_0603Metric, F.Cu at (117.6, 128.7)
- added R28: 221, Resistor_SMD:R_0201_0603Metric, F.Cu at (117.6, 130.4)
- added R29: 221, Resistor_SMD:R_0201_0603Metric, F.Cu at (117.6, 132.2)
- added R30: 221, Resistor_SMD:R_0201_0603Metric, F.Cu at (117.6, 133.9)
- added R31: 103, Resistor_SMD:R_0201_0603Metric, F.Cu at (120.1, 128.7)
- added R32: 103, Resistor_SMD:R_0201_0603Metric, F.Cu at (120.1, 130.4)
- added R33: 103, Resistor_SMD:R_0201_0603Metric, F.Cu at (120.1, 132.2)
- added R34: 103, Resistor_SMD:R_0201_0603Metric, F.Cu at (120.1, 133.9)
- added Y2: Crystal, Crystal:Crystal_HC35-U, F.Cu at (145.3, 123.5)
- IC2: footprint footprints:SOIC127P600X175-8N -> footprints:EEPROM
- J1, J16, J17: footprint Connector_PinHeader_1.00mm:PinHeader_1x05_P1.00mm_Vertical -> Connector_PinHeader_2.54mm:PinHeader_1x05_P2.54mm_Vertical
- J15: footprint Connector_PinHeader_2.00mm:PinHeader_1x03_P2.00mm_Vertical -> Connector_PinHeader_2.54mm:PinHeader_1x03_P2.54mm_Vertical
- J4: value Conn_02x16_Odd_Even -> Conn_01x04; footprint Connector_PinHeader_2.54mm:PinHeader_2x16_P2.54mm_Vertical -> Connector_PinHeader_2.54mm:PinHeader_1x04_P2.54mm_Vertical
- J6, J8: value Conn_02x16_Odd_Even -> Conn_01x03; footprint Connector_PinHeader_2.54mm:PinHeader_2x16_P2.54mm_Vertical -> Connector_PinHeader_2.54mm:PinHeader_1x03_P2.54mm_Vertical
- J7: value Conn_02x16_Odd_Even -> Conn_01x02; footprint Connector_PinHeader_2.54mm:PinHeader_2x16_P2.54mm_Vertical -> Connector_PinHeader_2.54mm:PinHeader_1x02_P2.54mm_Vertical
- R1: value 10k -> 100
- R14: value 103 -> R
- R2: value 10k -> R
- moved J7 142.4 mm to (26.1, 142.8)
- moved J6 128.4 mm to (16.8, 142.8)
- moved J4 127.8 mm to (138.3, 67.7)
- moved DS1 127.1 mm to (48.5, 43.1)
- moved J8 123.1 mm to (21.4, 142.8)
- moved D1 113.6 mm to (120.0, 21.6)
- moved D2 113.6 mm to (120.0, 27.5)
- moved D7 113.6 mm to (139.8, 21.6)
- moved D8 113.6 mm to (139.8, 27.5)
- moved D3 113.6 mm to (126.6, 21.6)
- moved D4 113.6 mm to (126.6, 27.5)
- moved D5 113.6 mm to (133.2, 21.6)
- moved D6 113.6 mm to (133.2, 27.5)
- moved J2 113.6 mm to (111.9, 21.0)
- moved R10 113.6 mm to (115.4, 31.8)
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Connections:
- net /Zegar czasu rzeczywistego RTC/SCL renamed Net-(IC1-SCL)
- net /Zegar czasu rzeczywistego RTC/SDA renamed Net-(IC1-SDA)
- J4 pad 1: /c1 -> Net-(J4-Pin_1)
- J4 pad 2: /c1 -> Net-(IC5-CLK)
- J4 pad 3: /c2 -> Net-(IC5-DOUT)
- J4 pad 4: /c2 -> Net-(IC5-DIN)
- J6 pad 1: /a1 -> Net-(J6-Pin_1)
- J6 pad 2: /a1 -> Net-(J6-Pin_2)
- J6 pad 3: /a2 -> Net-(J6-Pin_3)
- J7 pad 1: /b1 -> Net-(J7-Pin_1)
- J7 pad 2: /b1 -> Net-(J7-Pin_2)
- J8 pad 1: /d1 -> Net-(J8-Pin_1)
- J8 pad 2: /d1 -> Net-(J8-Pin_2)
- J8 pad 3: /d2 -> Net-(J8-Pin_3)
- R1 pad 1: Net-(U2-SDA) -> +3.3V
- R1 pad 2: +3.3V -> Net-(DS1-LED-A)
- R14 pad 1: +3.3V -> Net-(J13-Pin_2)
- R14 pad 2: /czujnik temperatury/czujnik temperatury -> Net-(U2B-P1W)
- R2 pad 2: +3.3V -> Net-(U2A-P0W)
