File: board_src/board.kicad_pcb (KiCad board)
At the start: 2 copper layers, 103 parts, among them IC1 PCF8563TS_4,118, IC2 M24C02-WMN6TP, IC3 DS18B20+, IC4 LM317T, IC5 MCP3202-CI_MS, J1 Conn_01x05, J10 Conn_01x01_Pin, J11 Conn_01x03, J12 112J-TDAR-R01, J13 Conn_01x03, J14 Conn_01x07, J15 Conn_01x03, J16 Conn_01x05, J17 Conn_01x05, J18 Conn_02x20_Counter_Clockwise, J19 USB_C_Receptacle_PowerOnly_6P, J2 Conn_01x08, J20 Conn_02x20_Counter_Clockwise, J21 Conn_02x20_Counter_Clockwise, J22 Conn_02x20_Counter_Clockwise, J23 Conn_01x04, J24 Conn_01x08, J25 Conn_01x04, J3 Conn_01x06, J4 Conn_01x04, J5 Conn_01x08, J6 Conn_01x03, J7 Conn_01x02, J8 Conn_01x03, J9 Conn_01x02_Pin, Q1 NPN, Q2 SS8550, Q3 SS8550, Q4 SS8550, Q5 SS8550, SW1 SW_Push, SW2 SW_Push, U1 Pico, U2 MCP4431-xxxx-ST, U4 Pico, Y2 Crystal

Commit message: wersja 3d
Parts:
- removed SW1, SW2: SW_Push, Button_Switch_THT:SW_PUSH_6mm
- removed SW10, SW3, SW4, SW5, SW6, SW7, SW8, SW9: ~, Button_Switch_THT:SW_PUSH_6mm
- removed U2: MCP4431-xxxx-ST, Package_SO:TSSOP-20_4.4x6.5mm_P0.65mm
- added S1: 1301.9319, footprints:przycisk, F.Cu at (108.7, 73.1)
- added S10: 1301.9319, footprints:przycisk, F.Cu at (109.7, 109.5)
- added S2: 1301.9319, footprints:przycisk, F.Cu at (117.1, 73.1)
- added S3: 1301.9319, footprints:przycisk, F.Cu at (52.9, 109.5)
- added S4: 1301.9319, footprints:przycisk, F.Cu at (61.0, 109.5)
- added S5: 1301.9319, footprints:przycisk, F.Cu at (69.1, 109.5)
- added S6: 1301.9319, footprints:przycisk, F.Cu at (77.2, 109.5)
- added S7: 1301.9319, footprints:przycisk, F.Cu at (85.3, 109.5)
- added S8: 1301.9319, footprints:przycisk, F.Cu at (93.5, 109.5)
- added S9: 1301.9319, footprints:przycisk, F.Cu at (101.6, 109.5)
- added VR1: PT6KV-251A2020, footprints:PT6KV251A2020, F.Cu at (139.2, 114.3)
- added VR2: PT6KV-251A2020, footprints:PT6KV251A2020, F.Cu at (148.7, 114.3)
- J13: footprint Connector_PinHeader_2.54mm:PinHeader_1x13_P2.54mm_Vertical -> Connector_PinHeader_2.54mm:PinHeader_1x03_P2.54mm_Vertical
- J7: value Conn_01x02 -> Conn_01x16; footprint Connector_PinHeader_2.54mm:PinHeader_1x02_P2.54mm_Vertical -> Connector_PinSocket_2.54mm:PinSocket_1x16_P2.54mm_Vertical
- Y2: footprint Crystal:Crystal_HC35-U -> Crystal:Crystal_AT310_D3.0mm_L10.0mm_Horizontal
- moved J3 245.4 mm to (259.8, 36.3)
- moved R1 197.9 mm to (215.8, 99.3)
- moved J7 166.9 mm to (178.1, 73.9), turned to 90 degrees
- moved D12 149.8 mm to (44.5, 40.9)
- moved DS1 149.6 mm to (198.1, 42.2)
- moved C1 149.2 mm to (41.7, 41.1)
- moved D13 149.2 mm to (44.7, 43.9)
- moved C2 148.2 mm to (42.0, 43.9)
- moved R17 146.6 mm to (42.0, 47.8)
- moved R18 146.6 mm to (42.0, 49.5)
- moved BT2 143.4 mm to (25.3, 52.8)
- moved J8 138.4 mm to (138.4, 68.8), turned to -90 degrees
- moved R11 137.1 mm to (21.1, 65.1), turned to 90 degrees
- moved R12 135.6 mm to (22.8, 65.1), turned to 90 degrees
- moved IC1 135.0 mm to (47.0, 48.8)
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Connections:
- J18 pad 10: /a10 -> /a5
- J18 pad 11: /a11 -> /a6
- J18 pad 12: /a12 -> /a6
- J18 pad 13: /a13 -> /a7
- J18 pad 14: /a14 -> /a7
- J18 pad 15: /a15 -> /a8
- J18 pad 16: /a16 -> /a8
- J18 pad 17: /a17 -> /a9
- J18 pad 18: /a18 -> /a9
- J18 pad 19: /a19 -> /a10
- J18 pad 2: /a2 -> /a1
- J18 pad 20: /a20 -> /a10
- J18 pad 21: /a20 -> /a11
- J18 pad 22: /a19 -> /a11
- J18 pad 23: /a18 -> /a12
- J18 pad 24: /a17 -> /a12
- J18 pad 25: /a16 -> /a13
- J18 pad 26: /a15 -> /a13
- J18 pad 28: /a13 -> /a14
- J18 pad 29: /a12 -> /a15
- J18 pad 3: /a3 -> /a2
- J18 pad 30: /a11 -> /a15
- J18 pad 31: /a10 -> /a16
- J18 pad 32: /a9 -> /a16
- J18 pad 33: /a8 -> /a17
- J18 pad 34: /a7 -> /a17
- J18 pad 35: /a6 -> /a18
- J18 pad 36: /a5 -> /a18
- J18 pad 37: /a4 -> /a19
- J18 pad 38: /a3 -> /a19
- J18 pad 39: /a2 -> /a20
- J18 pad 4: /a4 -> /a2
- J18 pad 40: /a1 -> /a20
- J18 pad 5: /a5 -> /a3
- J18 pad 6: /a6 -> /a3
- J18 pad 7: /a7 -> /a4
- J18 pad 8: /a8 -> /a4
- J18 pad 9: /a9 -> /a5
- J20 pad 10: /b10 -> /b5
- J20 pad 11: /b11 -> /b6
- J20 pad 12: /b12 -> /b6
- J20 pad 13: /b13 -> /b7
- J20 pad 14: /b14 -> /b7
- J20 pad 15: /b15 -> /b8
- J20 pad 16: /b16 -> /b8
- J20 pad 17: /b17 -> /b9
- J20 pad 18: /b18 -> /b9
- J20 pad 19: /b19 -> /b10
- J20 pad 2: /b2 -> /b1
- J20 pad 20: /b20 -> /b10
- J20 pad 21: /b20 -> /b11
- J20 pad 22: /b19 -> /b11
- J20 pad 23: /b18 -> /b12
- J20 pad 24: /b17 -> /b12
- J20 pad 25: /b16 -> /b13
- J20 pad 26: /b15 -> /b13
- J20 pad 28: /b13 -> /b14
- J20 pad 29: /b12 -> /b15
- J20 pad 3: /b3 -> /b2
- J20 pad 30: /b11 -> /b15
- J20 pad 31: /b10 -> /b16
- J20 pad 32: /b9 -> /b16
- J20 pad 33: /b8 -> /b17
- J20 pad 34: /b7 -> /b17
- J20 pad 35: /b6 -> /b18
- J20 pad 36: /b5 -> /b18
- J20 pad 37: /b4 -> /b19
- J20 pad 38: /b3 -> /b19
- J20 pad 39: /b2 -> /b20
- J20 pad 4: /b4 -> /b2
- J20 pad 40: /b1 -> /b20
- J20 pad 5: /b5 -> /b3
- J20 pad 6: /b6 -> /b3
- J20 pad 7: /b7 -> /b4
- J20 pad 8: /b8 -> /b4
- J20 pad 9: /b9 -> /b5
- J21 pad 10: /c10 -> /c5
- J21 pad 11: /c11 -> /c6
- J21 pad 12: /c12 -> /c6
- J21 pad 13: /c13 -> /c7
- J21 pad 14: /c14 -> /c7
- J21 pad 15: /c15 -> /c8
- J21 pad 16: /c16 -> /c8
- J21 pad 17: /c17 -> /c9
- J21 pad 18: /c18 -> /c9
- J21 pad 19: /c19 -> /c10
- J21 pad 2: /c2 -> /c1
- J21 pad 20: /c20 -> /c10
- J21 pad 21: /c20 -> /c11
- J21 pad 22: /c19 -> /c11
- J21 pad 23: /c18 -> /c12
- J21 pad 24: /c17 -> /c12
- J21 pad 25: /c16 -> /c13
- J21 pad 26: /c15 -> /c13
- J21 pad 28: /c13 -> /c14
- J21 pad 29: /c12 -> /c15
- J21 pad 3: /c3 -> /c2
- J21 pad 30: /c11 -> /c15
- J21 pad 31: /c10 -> /c16
- J21 pad 32: /c9 -> /c16
- J21 pad 33: /c8 -> /c17
- J21 pad 34: /c7 -> /c17
- J21 pad 35: /c6 -> /c18
- J21 pad 36: /c5 -> /c18
- J21 pad 37: /c4 -> /c19
- J21 pad 38: /c3 -> /c19
- J21 pad 39: /c2 -> /c20
- J21 pad 4: /c4 -> /c2
- J21 pad 40: /c1 -> /c20
- J21 pad 5: /c5 -> /c3
- J21 pad 6: /c6 -> /c3
- J21 pad 7: /c7 -> /c4
- J21 pad 8: /c8 -> /c4
- J21 pad 9: /c9 -> /c5
- J22 pad 10: /d10 -> /d5
- J22 pad 11: /d11 -> /d6
- J22 pad 12: /d12 -> /d6
- J22 pad 13: /d13 -> /d7
- J22 pad 14: /d14 -> /d7
- J22 pad 15: /d15 -> /d8
- J22 pad 16: /d16 -> /d8
- J22 pad 17: /d17 -> /d9
- J22 pad 18: /d18 -> /d9
- J22 pad 19: /d19 -> /d10
- J22 pad 2: /d2 -> /d1
- J22 pad 20: /d20 -> /d10
- J22 pad 21: /d20 -> /d11
- J22 pad 22: /d19 -> /d11
- J22 pad 23: /d18 -> /d12
- J22 pad 24: /d17 -> /d12
- J22 pad 25: /d16 -> /d13
- J22 pad 26: /d15 -> /d13
- J22 pad 28: /d13 -> /d14
- J22 pad 29: /d12 -> /d15
- J22 pad 3: /d3 -> /d2
- J22 pad 30: /d11 -> /d15
- J22 pad 31: /d10 -> /d16
- J22 pad 32: /d9 -> /d16
- J22 pad 33: /d8 -> /d17
- J22 pad 34: /d7 -> /d17
- J22 pad 35: /d6 -> /d18
- J22 pad 36: /d5 -> /d18
- J22 pad 37: /d4 -> /d19
- J22 pad 38: /d3 -> /d19
- J22 pad 39: /d2 -> /d20
- J22 pad 4: /d4 -> /d2
- J22 pad 40: /d1 -> /d20
- J22 pad 5: /d5 -> /d3
- J22 pad 6: /d6 -> /d3
- J22 pad 7: /d7 -> /d4
- J22 pad 8: /d8 -> /d4
- J22 pad 9: /d9 -> /d5
- J7 pad 1: Net-(J7-Pin_1) -> unconnected-(J7-Pin_1-Pad1)
- J7 pad 2: Net-(J7-Pin_2) -> unconnected-(J7-Pin_2-Pad2)
Routing:
- net Net-(D1-K): track 0.00 -> 13.5 mm
- net /b9: track 0.00 -> 11.4 mm
- net /b8: track 0.00 -> 11.4 mm
- net /b7: track 0.00 -> 11.4 mm
- net /b6: track 0.00 -> 11.4 mm
- net /b5: track 0.00 -> 11.4 mm
- net /b4: track 0.00 -> 11.4 mm
- net /b3: track 0.00 -> 11.4 mm
- net /b20: track 0.00 -> 11.4 mm
- net /b2: track 0.00 -> 11.4 mm
- net /b19: track 0.00 -> 11.4 mm
- net /b18: track 0.00 -> 11.4 mm
- net /b17: track 0.00 -> 11.4 mm
- net /b16: track 0.00 -> 11.4 mm
- net /b15: track 0.00 -> 11.4 mm
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
Commit message: uporzadkowane 3D
Parts:
- removed C3: 1n, Capacitor_SMD:C_0201_0603Metric
- removed D14: 1N4007, Diode_THT:D_DO-41_SOD81_P10.16mm_Horizontal
- removed IC4: LM317T, footprints:TO255P460X1020X2008-3P
- removed R11, R12: 5.1k, Resistor_SMD:R_0201_0603Metric
- added J26: Conn_01x16, Connector_PinHeader_2.54mm:PinHeader_1x16_P2.54mm_Vertical, F.Cu at (188.0, 79.5)
- added J27: USB4135-GF-A, footprints:USB4135GFA, F.Cu at (17.3, 20.6)
- added J28: Conn_01x01_Pin, Connector_PinHeader_2.54mm:PinHeader_1x01_P2.54mm_Vertical, F.Cu at (35.6, 23.9)
- added PS1: AP2202K-3.3TRG1, footprints:SOT95P282X145-5N, F.Cu at (179.1, 40.4)
- added R35: 5.1k, Resistor_SMD:R_0201_0603Metric, F.Cu at (17.4, 29.5)
- added R36: 5.1k, Resistor_SMD:R_0201_0603Metric, F.Cu at (19.2, 29.5)
- J19: value USB_C_Receptacle_PowerOnly_6P -> Conn_01x01_Pin; footprint Connector_USB:USB_C_Receptacle_GCT_USB4135-GF-A_6P_TopMnt_Horizontal -> Connector_PinHeader_2.54mm:PinHeader_1x01_P2.54mm_Vertical
- R15, R16: value 10k -> 4.7k
- moved J14 160.5 mm to (178.6, 34.9)
- moved J12 160.5 mm to (185.9, 21.9)
- moved J3 158.8 mm to (107.4, 80.8)
- moved DS1 158.2 mm to (46.4, 87.4)
- moved R21 74.3 mm to (65.8, 59.0)
- moved R22 74.3 mm to (64.0, 59.0)
- moved R23 74.1 mm to (64.6, 56.2)
- moved J15 73.2 mm to (55.9, 52.1)
- moved LED1 72.3 mm to (58.4, 59.4)
- moved J11 62.8 mm to (70.9, 52.6), turned to 90 degrees
- moved R10 57.5 mm to (18.8, 46.6)
- moved R3 57.5 mm to (40.5, 46.5)
- moved R4 57.5 mm to (39.8, 46.5)
- moved R5 57.5 mm to (39.0, 46.5)
- moved R6 57.5 mm to (38.2, 46.5)
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Connections:
- J7 pad 1: unconnected-(J7-Pin_1-Pad1) -> Net-(J26-Pin_16)
- J7 pad 10: unconnected-(J7-Pin_10-Pad10) -> Net-(J26-Pin_7)
- J7 pad 11: unconnected-(J7-Pin_11-Pad11) -> Net-(J26-Pin_6)
- J7 pad 12: unconnected-(J7-Pin_12-Pad12) -> Net-(J26-Pin_5)
- J7 pad 13: unconnected-(J7-Pin_13-Pad13) -> Net-(J26-Pin_4)
- J7 pad 14: unconnected-(J7-Pin_14-Pad14) -> Net-(J26-Pin_3)
- J7 pad 15: unconnected-(J7-Pin_15-Pad15) -> Net-(J26-Pin_2)
- J7 pad 16: unconnected-(J7-Pin_16-Pad16) -> Net-(J26-Pin_1)
- J7 pad 2: unconnected-(J7-Pin_2-Pad2) -> Net-(J26-Pin_15)
- J7 pad 3: unconnected-(J7-Pin_3-Pad3) -> Net-(J26-Pin_14)
- J7 pad 4: unconnected-(J7-Pin_4-Pad4) -> Net-(J26-Pin_13)
- J7 pad 5: unconnected-(J7-Pin_5-Pad5) -> Net-(J26-Pin_12)
- J7 pad 6: unconnected-(J7-Pin_6-Pad6) -> Net-(J26-Pin_11)
- J7 pad 7: unconnected-(J7-Pin_7-Pad7) -> Net-(J26-Pin_10)
- J7 pad 8: unconnected-(J7-Pin_8-Pad8) -> Net-(J26-Pin_9)
- J7 pad 9: unconnected-(J7-Pin_9-Pad9) -> Net-(J26-Pin_8)
- R15 pad 2: +3.3V -> Net-(J19-Pin_1)
- R16 pad 2: +3.3V -> Net-(J28-Pin_1)
Routing:
- net Net-(J5-Pin_8): track 0.00 -> 30.7 mm
- net Net-(J5-Pin_1): track 0.00 -> 25.1 mm
- net Net-(J5-Pin_7): track 0.00 -> 24.4 mm
- net Net-(J5-Pin_2): track 0.00 -> 19.7 mm
- net Net-(J5-Pin_6): track 0.00 -> 18.3 mm
- net Net-(J5-Pin_5): track 0.00 -> 14.1 mm
- net Net-(J5-Pin_3): track 0.00 -> 13.6 mm
- net Net-(J5-Pin_4): track 0.00 -> 10.6 mm
- net /Gniazdo kart micro SD/m1: track 0.15 -> 9.46 mm
- net /Gniazdo kart micro SD/m2: track 0.00 -> 7.97 mm
- net /Gniazdo kart micro SD/m3: track 0.00 -> 6.68 mm
- net /Gniazdo kart micro SD/m4: track 0.00 -> 6.49 mm
- net /Gniazdo kart micro SD/m5: track 0.00 -> 6.35 mm
- net /Gniazdo kart micro SD/m7: track 0.00 -> 6.25 mm
- net /Gniazdo kart micro SD/m6: track 0.00 -> 5.75 mm
Other:
- board text added: "EEPROM"
- board text added: "LEDS"
- board text added: "R G B"
- board text added: "RESET"
- board text added: "SWITCHS"

Commit message: wersja z wyswietlaczem LCD
Parts:
- removed BT2: 502-3, footprints:podstawka_bateria
- removed D1, D3, D5, D7: red, footprints:L128GRN2003500000
- removed D2, D4, D6, D8: green, footprints:L128GRN2003500000
- removed J26: Conn_01x16, Connector_PinHeader_2.54mm:PinHeader_1x16_P2.54mm_Vertical
- removed J28: Conn_01x01_Pin, Connector_PinHeader_2.54mm:PinHeader_1x01_P2.54mm_Vertical
- removed J7: Conn_01x16, Connector_PinSocket_2.54mm:PinSocket_1x16_P2.54mm_Vertical
- removed R10, R4, R6, R8: 122, Resistor_SMD:R_0201_0603Metric
- removed R5, R7, R9: 221, Resistor_SMD:R_0201_0603Metric
- added BT1: 3012, footprints:3012, B.Cu at (-2.68, 42.0)
- added C3: 10uF, Capacitor_SMD:C_0201_0603Metric, F.Cu at (178.6, 40.8)
- added C5: 100uF, Capacitor_SMD:C_0201_0603Metric, F.Cu at (178.6, 40.0)
- added C6: 100uF, Capacitor_SMD:C_0201_0603Metric, F.Cu at (193.9, 40.8)
- added C7: 10uF, Capacitor_SMD:C_0201_0603Metric, F.Cu at (193.9, 40.0)
- added DS4: RC1602B-BIW-ESX, footprints:RC1602BBIWESX, F.Cu at (211.5, 79.2)
- added J29: Conn_01x08, Connector_PinHeader_2.54mm:PinHeader_1x08_P2.54mm_Vertical, F.Cu at (56.0, 61.2)
- added J30: Conn_01x05, Connector_PinHeader_2.54mm:PinHeader_1x05_P2.54mm_Vertical, F.Cu at (180.8, 52.6)
- added J31: Conn_01x05, Connector_PinHeader_2.54mm:PinHeader_1x05_P2.54mm_Vertical, F.Cu at (181.1, 46.1)
- added LED2: red, footprints:LEDC1608X80N, F.Cu at (73.8, 56.0)
- added LED3: red, footprints:LEDC1608X80N, F.Cu at (68.7, 56.0)
- added LED4: red, footprints:LEDC1608X80N, F.Cu at (63.6, 56.0)
- added LED5: red, footprints:LEDC1608X80N, F.Cu at (58.5, 56.2)
- added LED6: green, footprints:LEDC1608X100N, F.Cu at (71.2, 56.0)
- added LED7: green, footprints:LEDC1608X100N, F.Cu at (66.2, 56.0)
- added LED8: green, footprints:LEDC1608X100N, F.Cu at (61.1, 56.2)
- added LED9: green, footprints:LEDC1608X100N, F.Cu at (56.0, 56.2)
- added Q6: BC107, OptoDevice:Osram_SFH3710, F.Cu at (259.1, 126.9)
- added R11: 68, Resistor_SMD:R_0201_0603Metric, F.Cu at (71.2, 51.8)
- added R12: 68, Resistor_SMD:R_0201_0603Metric, F.Cu at (70.5, 51.8)
- added R37: 68, Resistor_SMD:R_0201_0603Metric, F.Cu at (69.7, 51.8)
- added R38: 68, Resistor_SMD:R_0201_0603Metric, F.Cu at (68.9, 51.8)
- added R39: 68, Resistor_SMD:R_0201_0603Metric, F.Cu at (60.8, 51.1)
- added R40: 68, Resistor_SMD:R_0201_0603Metric, F.Cu at (60.1, 51.1)
- added R41: 68, Resistor_SMD:R_0201_0603Metric, F.Cu at (59.3, 51.2)
- added R42: 68, Resistor_SMD:R_0201_0603Metric, F.Cu at (58.5, 51.2)
- added RV1: R_Potentiometer, Potentiometer_SMD:Potentiometer_Bourns_3314R-GM5_Vertical, F.Cu at (260.0, 120.9)
- J19: value Conn_01x01_Pin -> Conn_02x07_Odd_Even; footprint Connector_PinHeader_2.54mm:PinHeader_1x01_P2.54mm_Vertical -> Connector_PinHeader_2.54mm:PinHeader_2x07_P2.54mm_Vertical
- J2: value Conn_01x08 -> Conn_01x05; footprint Connector_PinHeader_2.54mm:PinHeader_1x08_P2.54mm_Vertical -> Connector_PinHeader_2.54mm:PinHeader_1x05_P2.54mm_Vertical
- Q1: footprint Transistor_Power:GaN_Systems_GaNPX-3_5x6.6mm_Drain2.93x0.6mm -> OptoDevice:Osram_SFH3710
- R14, R2: value R -> 270
- R17, R18: value 10k -> 4.7k
- R20: value R -> 450
- R21, R22, R23: value 221 -> 68
- R3: value 221 -> R
- moved R3 232.6 mm to (257.9, 129.2), turned to 0 degrees
- moved J19 225.5 mm to (234.7, 125.1), turned to 90 degrees
- moved J2 157.7 mm to (180.8, 59.1)
- moved R19 122.0 mm to (79.5, 13.3)
- moved R1 82.4 mm to (111.0, 87.5)
- moved Q4 47.8 mm to (182.1, 116.3), turned to 180 degrees
- moved Q3 45.0 mm to (178.1, 116.3), turned to 180 degrees
- moved Q2 42.6 mm to (174.2, 116.3), turned to 180 degrees
- moved R28 42.1 mm to (157.7, 119.8)
- moved IC1 41.3 mm to (62.7, 40.6)
- moved R15 40.4 mm to (72.1, 19.7)
- moved R16 40.4 mm to (72.1, 20.4)
- moved IC3 40.1 mm to (79.5, 17.5), turned to 0 degrees
- moved IC2 39.7 mm to (65.7, 17.4)
- moved J9 38.2 mm to (64.0, 36.3)
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Connections:
- net /Wyświetlacz LED/DIG1 renamed /Wyświetlacz segmentowy/DIG1
- net /Wyświetlacz LED/DIG2 renamed /Wyświetlacz segmentowy/DIG2
- net /Wyświetlacz LED/DIG3 renamed /Wyświetlacz segmentowy/DIG3
- net /Wyświetlacz LED/DIG4 renamed /Wyświetlacz segmentowy/DIG4
- net /Wyświetlacz LED/DP renamed /Wyświetlacz segmentowy/DP
- net /Wyświetlacz LED/a renamed /Wyświetlacz segmentowy/a
- net /Wyświetlacz LED/b renamed /Wyświetlacz segmentowy/b
- net /Wyświetlacz LED/c renamed /Wyświetlacz segmentowy/c
- net /Wyświetlacz LED/d renamed /Wyświetlacz segmentowy/d
- net /Wyświetlacz LED/e renamed /Wyświetlacz segmentowy/e
- net /Wyświetlacz LED/f renamed /Wyświetlacz segmentowy/f
- net /Wyświetlacz LED/g renamed /Wyświetlacz segmentowy/g
- J15 pad 1: Net-(J15-Pin_1) -> Net-(J15-Pin_3)
- J15 pad 3: Net-(J15-Pin_3) -> Net-(J15-Pin_1)
- J19 pad 1: Net-(J19-Pin_1) -> /Wyświetlacz LCD/R/W
- J2 pad 1: Net-(D1-K) -> GND
- J2 pad 2: Net-(D8-K) -> GND
- J2 pad 3: Net-(D7-K) -> GND
- J2 pad 4: Net-(D6-K) -> GND
- J2 pad 5: Net-(D5-K) -> GND
- R15 pad 2: Net-(J19-Pin_1) -> +3.3V
- R16 pad 2: Net-(J28-Pin_1) -> +3.3V
- R3 pad 1: +3.3V -> Net-(Q6-B)
- R3 pad 2: Net-(D2-A) -> /Wyświetlacz LCD/BL
Routing:
- net Net-(D1-K): track 13.5 -> 0.00 mm
- net Net-(D1-A): track 10.6 -> 0.00 mm
- net Net-(D6-A): track 10.3 -> 0.00 mm
- net Net-(D5-A): track 10.2 -> 0.00 mm
- net Net-(D2-A): track 9.96 -> 0.00 mm
- net Net-(Q5-B): track 0.00 -> 7.83 mm
- net Net-(D4-A): track 6.25 -> 0.00 mm
- net Net-(D8-A): track 6.19 -> 0.00 mm
- net Net-(J24-Pin_8): track 0.00 -> 6.12 mm
- net GND: track 0.00 -> 6.11 mm
- net Net-(D7-A): track 6.08 -> 0.00 mm
- net Net-(Q2-B): track 0.00 -> 6.06 mm
- net Net-(D3-A): track 6.04 -> 0.00 mm
- net Net-(J24-Pin_4): track 0.00 -> 5.97 mm
- net Net-(J24-Pin_1): track 0.00 -> 5.97 mm
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Other:
- board text added: "+3.3V"
- board text added: "+5.0V"
- board text added: "1"
- board text added: "1 2 3 4"
- board text added: "2"
- board text added: "CLK"
- board text added: "DIGIT"
- board text added: "DP G F E D C B A"
- board text added: "DS18B20+"
- board text added: "GND"
- board text added: "INT"
- board text added: "PCF8563"
- board text added: "POT"
- board text added: "SEGMENT"
- board text added: "SWITCHES"
- board text added: "WC"
- board text removed: "SWITCHS"
