File: board_src/board.kicad_pcb (KiCad board)
At the start: 2 copper layers, 220 x 150 mm, 163 parts, among them IC1 DS18B20+, IC2 M24C02-WMN6TP, IC3 FT232RNL-TUBE, IC4 MCP3202, IC5 MCP4921-E_P, J1 Conn_02x20_Counter_Clockwise, J10 Conn_01x05, J11 Conn_01x05, J12 Conn_01x05, J13 Conn_02x20_Counter_Clockwise, J14 Conn_02x20_Counter_Clockwise, J15 Conn_01x20_Socket, J16 Conn_01x20_Socket, J17 Conn_01x01_Pin, J18 Conn_01x01_Pin, J19 Conn_01x01_Pin, J2 Conn_01x20_Socket, J20 Conn_02x20_Counter_Clockwise, J21 Conn_01x03, J22 Conn_01x02_Pin, J23 Conn_01x02_Pin, J24 Conn_01x06, J25 Conn_01x02_Pin, J26 Conn_01x02_Pin, J27 Battery, J28 Conn_01x07, J29 112J-TDAR-R01, J3 Conn_01x20_Socket, J30 Conn_01x03, J31 Conn_01x03, J32 Conn_02x05_Odd_Even, J33 USB_C_Receptacle_USB2.0_16P, J34 Conn_01x08, J35 Conn_01x04, J36 Conn_01x04, J37 Conn_01x08, J38 Conn_01x04, J39 Conn_01x08, J4 Conn_01x05, J40 Conn_01x16_Socket, J41 Conn_02x07_Odd_Even, J42 Conn_01x04, J43 Conn_01x04, J5 Conn_01x05, J6 Conn_01x05, J7 Conn_01x01_Pin, J8 Conn_01x01_Pin, J9 Conn_01x01_Pin, Q1 BSS123, Q2 SS8050-L, Q3 SS8550-L, Q4 SS8550-L, Q5 SS8550-L, Q6 SS8550-L, Q7 SS8050-L, U1 PCF8563TS, Y1 32.768kHz

Commit message: Naniesione poprawki na projekcie płytki. Wersja końcowa
Parts:
- added H5: MountingHole, MountingHole:MountingHole_2.7mm_M2.5, F.Cu at (73.8, 68.8)
- added H6: MountingHole, MountingHole:MountingHole_2.7mm_M2.5, F.Cu at (148.8, 68.8)
- added H7: MountingHole, MountingHole:MountingHole_2.7mm_M2.5, F.Cu at (73.8, 99.8)
- added H8: MountingHole, MountingHole:MountingHole_2.7mm_M2.5, F.Cu at (148.8, 99.8)
- R3: value 220 -> 470
- moved R52 34.7 mm to (85.0, 63.5)
- moved J27 24.3 mm to (90.0, 62.5), turned to 90 degrees
- moved D4 17.8 mm to (109.0, 59.5), turned to 90 degrees
- moved C10 11.4 mm to (207.2, 42.8), turned to 90 degrees
- moved IC3 9.46 mm to (22.0, 17.2), turned to 90 degrees
- moved R10 8.53 mm to (95.2, 53.8), turned to -90 degrees
- moved J43 7.08 mm to (210.0, 39.0)
- moved C9 7.04 mm to (198.2, 36.5), turned to 0 degrees
- moved D3 6.67 mm to (101.0, 62.0), turned to 180 degrees
- moved Q7 6.54 mm to (121.0, 75.2), turned to 180 degrees
- moved LED8 5.96 mm to (33.0, 17.2)
- moved R30 5.96 mm to (35.0, 17.2)
- moved LED7 5.96 mm to (28.9, 17.2)
- moved R29 5.96 mm to (30.9, 17.2)
- moved J42 4.48 mm to (192.2, 39.0), turned to 0 degrees
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Connections:
- net Net-(IC3-USBDM) renamed /Port USB/USBD-
- net Net-(IC3-USBDP) renamed /Port USB/USBD+
- J1 pad 15: /a8 -> GND
- J1 pad 16: /a8 -> GND
- J1 pad 25: /a13 -> GND
- J1 pad 26: /a13 -> GND
- J1 pad 35: /a18 -> GND
- J1 pad 36: /a18 -> GND
- J1 pad 5: /a3 -> GND
- J1 pad 6: /a3 -> GND
- J13 pad 15: /b8 -> GND
- J13 pad 16: /b8 -> GND
- J13 pad 25: /b13 -> GND
- J13 pad 26: /b13 -> GND
- J13 pad 3: +5.0V -> /VSYS
- J13 pad 35: /b18 -> GND
- J13 pad 36: /b18 -> GND
- J13 pad 4: +5V -> /VSYS
- J13 pad 5: /b3 -> GND
- J13 pad 6: /b3 -> GND
- J14 pad 15: /c8 -> GND
- J14 pad 16: /c8 -> GND
- J14 pad 25: /c13 -> GND
- J14 pad 26: /c13 -> GND
- J14 pad 35: /c18 -> GND
- J14 pad 36: /c18 -> GND
- J14 pad 5: /c3 -> GND
- J14 pad 6: /c3 -> GND
- J15 pad 13: /c13 -> GND
- J15 pad 18: /c18 -> GND
- J15 pad 3: /c3 -> GND
- J15 pad 8: /c8 -> GND
- J16 pad 13: /d8 -> GND
- J16 pad 18: /d3 -> GND
- J16 pad 19: +5V -> /VSYS_2
- J16 pad 3: /d18 -> GND
- J16 pad 8: /d13 -> GND
- J2 pad 13: /a13 -> GND
- J2 pad 18: /a18 -> GND
- J2 pad 3: /a3 -> GND
- J2 pad 8: /a8 -> GND
- J20 pad 15: /d8 -> GND
- J20 pad 16: /d8 -> GND
- J20 pad 25: /d13 -> GND
- J20 pad 26: /d13 -> GND
- J20 pad 3: +5V -> /VSYS_2
- J20 pad 35: /d18 -> GND
- J20 pad 36: /d18 -> GND
- J20 pad 4: +5V -> /VSYS_2
- J20 pad 5: /d3 -> GND
- J20 pad 6: /d3 -> GND
- J23 pad 1: Net-(IC2-SCL) -> Net-(IC2-SDA)
- J23 pad 2: Net-(IC2-SDA) -> Net-(IC2-SCL)
- J3 pad 13: /b8 -> GND
- J3 pad 18: /b3 -> GND
- J3 pad 19: +5V -> /VSYS
- J3 pad 3: /b18 -> GND
- J3 pad 8: /b13 -> GND
- J35 pad 1: GND -> Net-(IC4-~{CS}/SHDN)
- J35 pad 2: Net-(IC4-CH1) -> Net-(IC4-CH0)
- J35 pad 3: Net-(IC4-CH0) -> Net-(IC4-CH1)
- J35 pad 4: Net-(IC4-~{CS}/SHDN) -> GND
- J42 pad 1: Net-(IC5-SDI) -> Net-(IC5-VDD)
- J42 pad 2: Net-(IC5-SCK) -> Net-(IC5-~{CS})
- J42 pad 3: Net-(IC5-~{CS}) -> Net-(IC5-SCK)
- J42 pad 4: Net-(IC5-VDD) -> Net-(IC5-SDI)
- LED5 pad 1: Net-(J31-Pin_3) -> Net-(J31-Pin_1)
- LED5 pad 3: Net-(J31-Pin_1) -> Net-(J31-Pin_3)
Routing:
- net GND: track 1399.2 -> 1904.5 mm, vias 30 -> 47
- net +3.3V: track 643.4 -> 839.0 mm, vias 24 -> 15
- net +5V: track 416.6 -> 365.5 mm, vias 4 -> 2
- net Net-(S5-B): track 23.4 -> 50.1 mm
- net (no net): track 26.4 -> 0.00 mm, vias 14 -> 0
- net Net-(J40-Pin_15): track 6.48 -> 32.0 mm
- net Net-(D3-K): track 2.02 -> 20.5 mm, vias 0 -> 2
- net /Port USB/TXD: track 11.4 -> 27.5 mm
- net /Port USB/DTR: track 8.02 -> 22.7 mm
- net /Port USB/USBD+: track 23.3 -> 9.88 mm
- net /Port USB/RTS: track 11.3 -> 24.3 mm
- net /d11: track 40.7 -> 53.4 mm, vias 1 -> 0
- net /Port USB/USBD-: track 21.8 -> 9.39 mm
- net /VSYS: track 0.00 -> 11.5 mm
- net /b8: track 11.4 -> 0.00 mm
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Other:
- board text added: "+"
- board text added: "-"
- board text added: "3V3OUT"
- board text added: "8 7 6 5 4 3 2 1"
- board text added: "Bat"
- board text added: "DAT3"
- board text added: "DQ"
- board text added: "PCF 8563"
- board text removed: "3V3"
- board text removed: "CD/DAT3"
- board text removed: "RW"
- board text removed: "VCC"

Commit message: Wprowadzono usprawnienia i poprawki. Wersja ostateczna, wysłana do JLCPCB.
Parts:
- removed J19, J9: Conn_01x01_Pin, Connector_PinHeader_2.54mm:PinHeader_1x01_P2.54mm_Vertical
- added C11: 100n, Capacitor_SMD:C_0603_1608Metric_Pad1.08x0.95mm_HandSolder, F.Cu at (89.5, 130.8)
- added C12: 100n, Capacitor_SMD:C_0603_1608Metric_Pad1.08x0.95mm_HandSolder, F.Cu at (15.9, 24.2)
- added C13: 100n, Capacitor_SMD:C_0603_1608Metric_Pad1.08x0.95mm_HandSolder, F.Cu at (39.8, 14.2)
- added J44: Conn_01x02, Connector_PinHeader_2.54mm:PinHeader_1x02_P2.54mm_Vertical, F.Cu at (86.8, 134.2)
- J24: value Conn_01x06 -> Conn_01x07
- moved R2 3.93 mm to (183.2, 30.5), turned to 180 degrees
- moved LED2 3.85 mm to (179.2, 30.5), turned to 0 degrees
- moved LED3 2.77 mm to (173.0, 30.5)
- moved R3 2.65 mm to (169.8, 29.5), turned to -90 degrees
Connections:
- DS1 pad 10: +3.3V -> Net-(DS1-LED-A)
- DS1 pad 9: +3.3V -> Net-(DS1-LED-A)
Routing:
- net Net-(DS1-LED-A): track 0.00 -> 35.9 mm
- net GND: track 1904.5 -> 1929.1 mm
- net +3.3V: track 839.0 -> 824.0 mm
- net /Port USB/USBD+: track 9.88 -> 12.3 mm
- net /Port USB/USBD-: track 9.39 -> 11.2 mm
- net +5V: track 365.5 -> 366.6 mm
Other:
- board text added: "7-SEG DISPLAY"
- board text added: "ADC"
- board text added: "ALPHANUMERIC DISPLAY"
- board text added: "ALPHANUMERIC LCD (HD44780)"
- board text added: "BREADBOARD"
- board text added: "DAC"
- board text added: "GRAPHIC DISPLAY POWER JUMPER"
- board text added: "GRAPHICS DISPLAY"
- board text added: "LED RGB"
- board text added: "PICO-1"
- board text added: "PICO-2"
- board text added: "POTENTIOMETERS BUZZER"
- board text added: "RST"
- board text added: "Raspberry Pi PICO Module 1"
- board text added: "Raspberry Pi PICO Module 2"
- board text added: "Wyświetlacz alfanumeryczny"
- board text removed: "LCD"
- board text removed: "POT"
