File: board_src/microSD.kicad_sch (KiCad schematic)
At the start: 10 parts, among them J28 Conn_01x07, J29 112J-TDAR-R01

Commit message: Wprowadzono usprawnienia i poprawki. Wersja ostateczna, wysłana do JLCPCB.
Parts:
- J28: footprint Connector_PinHeader_2.54mm:PinHeader_1x04_P2.54mm_Vertical -> Connector_PinHeader_2.54mm:PinHeader_1x07_P2.54mm_Vertical
- J29: footprint Connector_PinHeader_2.54mm:PinHeader_1x08_P2.54mm_Vertical -> footprints:112JTDARR01
Changed lines of the file:
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@@
 			)
 		)
-		(property "Footprint" "Connector_PinHeader_2.54mm:PinHeader_1x08_P2.54mm_Vertical"
+		(property "Footprint" "footprints:112JTDARR01"
 			(at 143.51 188.9 0)
 			(effects
@@
 			)
 		)
-		(property "Footprint" "Connector_PinHeader_2.54mm:PinHeader_1x04_P2.54mm_Vertical"
+		(property "Footprint" "Connector_PinHeader_2.54mm:PinHeader_1x07_P2.54mm_Vertical"
 			(at 35.56 39.37 0)
 			(effects
