File: board_src/rgb.kicad_sch (KiCad schematic)
At the start: 5 parts, among them J31 Conn_01x03

Commit message: Wprowadzono usprawnienia i poprawki. Wersja ostateczna, wysłana do JLCPCB.
Parts:
- J31: footprint Connector_PinHeader_2.54mm:PinHeader_1x10_P2.54mm_Vertical -> Connector_PinHeader_2.54mm:PinHeader_1x03_P2.54mm_Vertical
- LED5: footprint LED_SMD:LED_0603_1608Metric_Pad1.05x0.95mm_HandSolder -> footprints:ASMT-YTC7-0AA02
Changed lines of the file:
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@@
 			)
 		)
-		(property "Footprint" "Connector_PinHeader_2.54mm:PinHeader_1x10_P2.54mm_Vertical"
+		(property "Footprint" "Connector_PinHeader_2.54mm:PinHeader_1x03_P2.54mm_Vertical"
 			(at 199.39 95.25 0)
 			(effects
@@
 			)
 		)
-		(property "Footprint" "LED_SMD:LED_0603_1608Metric_Pad1.05x0.95mm_HandSolder"
+		(property "Footprint" "footprints:ASMT-YTC7-0AA02"
 			(at 185.42 187.63 0)
 			(effects
