File: board_src/wyswietlaczlcd.kicad_sch (KiCad schematic)
At the start: 6 parts, among them J40 Conn_01x16_Socket, J41 Conn_02x07_Odd_Even, Q7 SS8050-L

Commit message: Naniesione poprawki na projekcie płytki. Wersja końcowa
Parts:
- added H5, H6, H7, H8: MountingHole, MountingHole:MountingHole_2.7mm_M2.5, symbol Mechanical:MountingHole
Other:
- note added: "Dla bezpieczeństwa połączony z masą, by porty wyświetlacza były zawsze wejściowe i napięcie +5V nie pojawiło się na pinach GPIO Raspberry Pi Pico"
- note added: "R/W"
- note removed: "Dla bezpieczeństwa, by porty wyświetlacza były zawsze wejściowe"
- moved on the sheet: J40, J41, Q7, R51, R52, RV1

Commit message: Wprowadzono usprawnienia i poprawki. Wersja ostateczna, wysłana do JLCPCB.
Parts:
- J40: footprint Connector_PinHeader_2.54mm:PinHeader_1x01_P2.54mm_Vertical -> Connector_PinSocket_2.54mm:PinSocket_1x16_P2.54mm_Vertical
- J41: footprint Connector_PinHeader_2.54mm:PinHeader_1x01_P2.54mm_Vertical -> Connector_PinHeader_2.54mm:PinHeader_2x07_P2.54mm_Vertical
Changed lines of the file:
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@@
 			)
 		)
-		(property "Footprint" "Connector_PinHeader_2.54mm:PinHeader_1x01_P2.54mm_Vertical"
+		(property "Footprint" "Connector_PinSocket_2.54mm:PinSocket_1x16_P2.54mm_Vertical"
 			(at 81.28 96.52 0)
 			(effects
@@
 			)
 		)
-		(property "Footprint" "Connector_PinHeader_2.54mm:PinHeader_1x01_P2.54mm_Vertical"
+		(property "Footprint" "Connector_PinHeader_2.54mm:PinHeader_2x07_P2.54mm_Vertical"
 			(at 132.08 111.76 0)
 			(effects
